File: BuckBoostTest/bb6v.kicad_sch (KiCad schematic)
At the start: 17 parts, among them U301 TPS63070RNMR

Commit message: BuckBoostTest v0.1
Parts:
- renumbered C301 to C201, C302 to C202, C303 to C203, C304 to C204, C305 to C205, C306 to C206, C307 to C207, C308 to C208, L301 to L201, R301 to R201, R302 to R202, R303 to R203, R304 to R204, TP301 to TP201, TP302 to TP202, TP303 to TP203, U301 to U201
Changed lines of the file:
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@@
 		(dnp no)
 		(fields_autoplaced yes)
-		(property "Reference" "R303"
+		(property "Reference" "R203"
 			(at 185.42 104.1399 0)
 			(effects
@@
 			(project ""
 				(path "/48ddfdd8-68fa-4e63-aa18-bc113cdf8cfa/35e7cf5c-95fe-496c-867d-9a2129f85874"
-					(reference "R303")
+					(reference "R203")
 					(unit 1)
 				)
@@
 		(dnp no)
 		(fields_autoplaced yes)
-		(property "Reference" "#PWR0301"
+		(property "Reference" "#PWR0201"
 			(at 78.74 104.14 0)
 			(effects
@@
 			(project ""
 				(path "/48ddfdd8-68fa-4e63-aa18-bc113cdf8cfa/35e7cf5c-95fe-496c-867d-9a2129f85874"
-					(reference "#PWR0301")
+					(reference "#PWR0201")
 					(unit 1)
 				)
@@
 		(dnp no)
 		(fields_autoplaced yes)
-		(property "Reference" "#PWR0308"
+		(property "Reference" "#PWR0208"
 			(at 173.99 127 0)
 			(effects
@@
 			(project ""
 				(path "/48ddfdd8-68fa-4e63-aa18-bc113cdf8cfa/35e7cf5c-95fe-496c-867d-9a2129f85874"
-					(reference "#PWR0308")
+					(reference "#PWR0208")
 					(unit 1)
 				)
@@
 		(dnp no)
 		(fields_autoplaced yes)
-		(property "Reference" "R304"
+		(property "Reference" "R204"
 			(at 195.58 105.4099 0)
 			(effects
@@
 			(project ""
 				(path "/48ddfdd8-68fa-4e63-aa18-bc113cdf8cfa/35e7cf5c-95fe-496c-867d-9a2129f85874"
-					(reference "R304")
+					(reference "R204")
 					(unit 1)
 				)
@@
 		(dnp no)
 		(fields_autoplaced yes)
-		(property "Reference" "U301"
+		(property "Reference" "U201"
 			(at 142.24 74.93 0)
 			(effects
@@
 			(project ""
 				(path "/48ddfdd8-68fa-4e63-aa18-bc113cdf8cfa/35e7cf5c-95fe-496c-867d-9a2129f85874"
-					(reference "U301")
+					(reference "U201")
 					(unit 1)
 				)
@@
 		(dnp no)
 		(fields_autoplaced yes)
-		(property "Reference" "TP303"
+		(property "Reference" "TP203"
 			(at 241.3 85.5979 0)
 			(effects
@@
 			(project "Blocks"
 				(path "/48ddfdd8-68fa-4e63-aa18-bc113cdf8cfa/35e7cf5c-95fe-496c-867d-9a2129f85874"
-					(reference "TP303")
+					(reference "TP203")
 					(unit 1)
 				)
@@
 		(dnp no)
 		(fields_autoplaced yes)
-		(property "Reference" "L301"
+		(property "Reference" "L201"
 			(at 143.51 63.5 90)
 			(effects
@@
 			(project ""
 				(path "/48ddfdd8-68fa-4e63-aa18-bc113cdf8cfa/35e7cf5c-95fe-496c-867d-9a2129f85874"
-					(reference "L301")
+					(reference "L201")
 					(unit 1)
 				)
@@
 		(dnp no)
 		(fields_autoplaced yes)
-		(property "Reference" "C302"
+		(property "Reference" "C202"
 			(at 93.98 92.7099 0)
 			(effects
@@
 			(project ""
 				(path "/48ddfdd8-68fa-4e63-aa18-bc113cdf8cfa/35e7cf5c-95fe-496c-867d-9a2129f85874"
-					(reference "C302")
+					(reference "C202")
 					(unit 1)
 				)
@@
 		(dnp no)
 		(fields_autoplaced yes)
-		(property "Reference" "#PWR0310"
+		(property "Reference" "#PWR0210"
 			(at 204.47 104.14 0)
 			(effects
@@
 			(project ""
 				(path "/48ddfdd8-68fa-4e63-aa18-bc113cdf8cfa/35e7cf5c-95fe-496c-867d-9a2129f85874"
-					(reference "#PWR0310")
+					(reference "#PWR0210")
 					(unit 1)
 				)
@@
 		(dnp no)
 		(fields_autoplaced yes)
-		(property "Reference" "R302"
+		(property "Reference" "R202"
 			(at 185.42 93.9799 0)
 			(effects
@@
 			(project ""
 				(path "/48ddfdd8-68fa-4e63-aa18-bc113cdf8cfa/35e7cf5c-95fe-496c-867d-9a2129f85874"
-					(reference "R302")
+					(reference "R202")
 					(unit 1)
 				)
@@
 		(dnp no)
 		(fields_autoplaced yes)
-		(property "Reference" "C308"
+		(property "Reference" "C208"
 			(at 232.41 92.7099 0)
 			(effects
@@
 			(project "Blocks"
 				(path "/48ddfdd8-68fa-4e63-aa18-bc113cdf8cfa/35e7cf5c-95fe-496c-867d-9a2129f85874"
-					(reference "C308")
+					(reference "C208")
 					(unit 1)
 				)
@@
 		(dnp no)
 		(fields_autoplaced yes)
-		(property "Reference" "C305"
+		(property "Reference" "C205"
 			(at 173.99 92.7099 0)
 			(effects
@@
 			(project "Blocks"
 				(path "/48ddfdd8-68fa-4e63-aa18-bc113cdf8cfa/35e7cf5c-95fe-496c-867d-9a2129f85874"
-					(reference "C305")
+					(reference "C205")
 					(unit 1)
 				)
@@
 		(dnp no)
 		(fields_autoplaced yes)
-		(property "Reference" "C307"
+		(property "Reference" "C207"
 			(at 220.98 92.7099 0)
 			(effects
@@
 			(project "Blocks"
 				(path "/48ddfdd8-68fa-4e63-aa18-bc113cdf8cfa/35e7cf5c-95fe-496c-867d-9a2129f85874"
-					(reference "C307")
+					(reference "C207")
 					(unit 1)
 				)
@@
 		(dnp no)
 		(fields_autoplaced yes)
-		(property "Reference" "#PWR0303"
+		(property "Reference" "#PWR0203"
 			(at 109.22 104.14 0)
 			(effects
@@
 			(project ""
 				(path "/48ddfdd8-68fa-4e63-aa18-bc113cdf8cfa/35e7cf5c-95fe-496c-867d-9a2129f85874"
-					(reference "#PWR0303")
+					(reference "#PWR0203")
 					(unit 1)
 				)
@@
 		(dnp no)
 		(fields_autoplaced yes)
-		(property "Reference" "TP302"
+		(property "Reference" "TP202"
 			(at 193.04 121.4119 0)
 			(effects
@@
 			(project ""
 				(path "/48ddfdd8-68fa-4e63-aa18-bc113cdf8cfa/35e7cf5c-95fe-496c-867d-9a2129f85874"
-					(reference "TP302")
+					(reference "TP202")
 					(unit 1)
 				)
@@
 		(dnp no)
 		(fields_autoplaced yes)
-		(property "Reference" "C301"
+		(property "Reference" "C201"
 			(at 82.55 92.7099 0)
 			(effects
@@
 			(project ""
 				(path "/48ddfdd8-68fa-4e63-aa18-bc113cdf8cfa/35e7cf5c-95fe-496c-867d-9a2129f85874"
-					(reference "C301")
+					(reference "C201")
 					(unit 1)
 				)
@@
 		(dnp no)
 		(fields_autoplaced yes)
-		(property "Reference" "C303"
+		(property "Reference" "C203"
 			(at 113.03 92.7099 0)
 			(effects
@@
 			(project ""
 				(path "/48ddfdd8-68fa-4e63-aa18-bc113cdf8cfa/35e7cf5c-95fe-496c-867d-9a2129f85874"
-					(reference "C303")
+					(reference "C203")
 					(unit 1)
 				)
@@
 		(dnp no)
 		(fields_autoplaced yes)
-		(property "Reference" "#PWR0305"
+		(property "Reference" "#PWR0205"
 			(at 114.3 104.14 0)
 			(effects
@@
 			(project "Blocks"
 				(path "/48ddfdd8-68fa-4e63-aa18-bc113cdf8cfa/35e7cf5c-95fe-496c-867d-9a2129f85874"
-					(reference "#PWR0305")
+					(reference "#PWR0205")
 					(unit 1)
 				)
@@
 		(dnp no)
 		(fields_autoplaced yes)
-		(property "Reference" "#PWR0302"
+		(property "Reference" "#PWR0202"
 			(at 90.17 104.14 0)
 			(effects
@@
 			(project ""
 				(path "/48ddfdd8-68fa-4e63-aa18-bc113cdf8cfa/35e7cf5c-95fe-496c-867d-9a2129f85874"
-					(reference "#PWR0302")
+					(reference "#PWR0202")
 					(unit 1)
 				)
@@
 		(dnp no)
 		(fields_autoplaced yes)
-		(property "Reference" "#PWR0307"
+		(property "Reference" "#PWR0207"
 			(at 171.45 124.46 0)
 			(effects
@@
 			(project "Blocks"
 				(path "/48ddfdd8-68fa-4e63-aa18-bc113cdf8cfa/35e7cf5c-95fe-496c-867d-9a2129f85874"
-					(reference "#PWR0307")
+					(reference "#PWR0207")
 					(unit 1)
 				)
@@
 		(dnp no)
 		(fields_autoplaced yes)
-		(property "Reference" "#PWR0306"
+		(property "Reference" "#PWR0206"
 			(at 171.45 115.57 0)
 			(effects
@@
 			(project "Blocks"
 				(path "/48ddfdd8-68fa-4e63-aa18-bc113cdf8cfa/35e7cf5c-95fe-496c-867d-9a2129f85874"
-					(reference "#PWR0306")
+					(reference "#PWR0206")
 					(unit 1)
 				)
@@
 		(dnp no)
 		(fields_autoplaced yes)
-		(property "Reference" "#PWR0309"
+		(property "Reference" "#PWR0209"
 			(at 170.18 104.14 0)
 			(effects
@@
 			(project ""
 				(path "/48ddfdd8-68fa-4e63-aa18-bc113cdf8cfa/35e7cf5c-95fe-496c-867d-9a2129f85874"
-					(reference "#PWR0309")
+					(reference "#PWR0209")
 					(unit 1)
 				)
@@
 		(dnp no)
 		(fields_autoplaced yes)
-		(property "Reference" "C304"
+		(property "Reference" "C204"
 			(at 118.11 129.5399 0)
 			(effects
@@
 			(project ""
 				(path "/48ddfdd8-68fa-4e63-aa18-bc113cdf8cfa/35e7cf5c-95fe-496c-867d-9a2129f85874"
-					(reference "C304")
+					(reference "C204")
 					(unit 1)
 				)
@@
 		(dnp no)
 		(fields_autoplaced yes)
-		(property "Reference" "C306"
+		(property "Reference" "C206"
 			(at 208.28 92.7099 0)
 			(effects
@@
 			(project "Blocks"
 				(path "/48ddfdd8-68fa-4e63-aa18-bc113cdf8cfa/35e7cf5c-95fe-496c-867d-9a2129f85874"
-					(reference "C306")
+					(reference "C206")
 					(unit 1)
 				)
@@
 		(dnp no)
 		(fields_autoplaced yes)
-		(property "Reference" "TP301"
+		(property "Reference" "TP201"
 			(at 76.2 85.5979 0)
 			(effects
@@
 			(project "Blocks"
 				(path "/48ddfdd8-68fa-4e63-aa18-bc113cdf8cfa/35e7cf5c-95fe-496c-867d-9a2129f85874"
-					(reference "TP301")
+					(reference "TP201")
 					(unit 1)
 				)
@@
 		(dnp no)
 		(fields_autoplaced yes)
-		(property "Reference" "R301"
+		(property "Reference" "R201"
 			(at 104.14 102.8699 0)
 			(effects
@@
 			(project ""
 				(path "/48ddfdd8-68fa-4e63-aa18-bc113cdf8cfa/35e7cf5c-95fe-496c-867d-9a2129f85874"
-					(reference "R301")
+					(reference "R201")
 					(unit 1)
 				)
@@
 		(dnp no)
 		(fields_autoplaced yes)
-		(property "Reference" "#PWR0304"
+		(property "Reference" "#PWR0204"
 			(at 114.3 144.78 0)
 			(effects
@@
 			(project "Blocks"
 				(path "/48ddfdd8-68fa-4e63-aa18-bc113cdf8cfa/35e7cf5c-95fe-496c-867d-9a2129f85874"
-					(reference "#PWR0304")
+					(reference "#PWR0204")
 					(unit 1)
 				)
@@
 		(dnp no)
 		(fields_autoplaced yes)
-		(property "Reference" "#PWR0312"
+		(property "Reference" "#PWR0212"
 			(at 228.6 104.14 0)
 			(effects
@@
 			(project ""
 				(path "/48ddfdd8-68fa-4e63-aa18-bc113cdf8cfa/35e7cf5c-95fe-496c-867d-9a2129f85874"
-					(reference "#PWR0312")
+					(reference "#PWR0212")
 					(unit 1)
 				)
@@
 		(dnp no)
 		(fields_autoplaced yes)
-		(property "Reference" "#PWR0311"
+		(property "Reference" "#PWR0211"
 			(at 217.17 104.14 0)
 			(effects
@@
 			(project ""
 				(path "/48ddfdd8-68fa-4e63-aa18-bc113cdf8cfa/35e7cf5c-95fe-496c-867d-9a2129f85874"
-					(reference "#PWR0311")
-					(unit 1)
-				)
+					(reference "#PWR0211")
+					(unit 1)
+				)

Commit message: revisions
Parts:
- TP201, TP202, TP203: now not fitted
Changed lines of the file:
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@@
 		(in_bom no)
 		(on_board yes)
-		(dnp no)
+		(dnp yes)
 		(fields_autoplaced yes)
 		(property "Reference" "TP203"
@@
 		(in_bom no)
 		(on_board yes)
-		(dnp no)
+		(dnp yes)
 		(fields_autoplaced yes)
 		(property "Reference" "TP202"
@@
 		(in_bom no)
 		(on_board yes)
-		(dnp no)
+		(dnp yes)
 		(fields_autoplaced yes)
 		(property "Reference" "TP201"
