File: BuckBoostTest/BuckBoostTest.kicad_pcb (KiCad board)
At the start: 4 copper layers, 99.5 x 61.2 mm, 36 parts, among them U101 MC7805CDTRKG, U102 ADM7150ARDZ-5.0, U201 TPS63070RNMR

Commit message: revisions
Parts:
- C101: value C -> 10uf
Changed lines of the file:
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@@
 		(sheetname "Root")
 		(sheetfile "BuckBoostTest.kicad_sch")
-		(attr through_hole)
+		(attr through_hole exclude_from_bom dnp)
 		(fp_text user "${REFERENCE}"
 			(at 0 2.5 0)
@@
 		(sheetname "BB6V")
 		(sheetfile "bb6v.kicad_sch")
-		(attr through_hole exclude_from_bom)
+		(attr through_hole exclude_from_bom dnp)
 		(fp_circle
 			(center 0 0)
@@
 		(sheetname "Root")
 		(sheetfile "BuckBoostTest.kicad_sch")
-		(attr through_hole)
+		(attr through_hole exclude_from_bom dnp)
 		(fp_text user "${REFERENCE}"
 			(at 0 2.5 0)
@@
 		(tags "capacitor")
 		(property "Reference" "C104"
-			(at 0 -1.5 360)
+			(at 0 -1.5 0)
 			(layer "F.SilkS")
 			(effects
@@
 		)
 		(property "Value" "10f"
-			(at 0 1.43 360)
+			(at 0 1.43 0)
 			(layer "F.Fab")
 			(effects
@@
 		)
 		(fp_text user "${REFERENCE}"
-			(at 0 0 360)
+			(at 0 0 0)
 			(layer "F.Fab")
 			(effects
@@
 		(tags "capacitor")
 		(property "Reference" "C103"
-			(at 3.5 0 360)
+			(at 3.5 0 0)
 			(layer "F.SilkS")
 			(effects
@@
 		)
 		(property "Value" "10uf"
-			(at 0 1.43 360)
+			(at 0 1.43 0)
 			(layer "F.Fab")
 			(effects
@@
 		)
 		(fp_text user "${REFERENCE}"
-			(at 0 0 360)
+			(at 0 0 0)
 			(layer "F.Fab")
 			(effects
@@
 		(sheetname "BB6V")
 		(sheetfile "bb6v.kicad_sch")
-		(attr through_hole exclude_from_bom)
+		(attr through_hole exclude_from_bom dnp)
 		(fp_circle
 			(center 0 0)
@@
 		(sheetname "Root")
 		(sheetfile "BuckBoostTest.kicad_sch")
-		(attr through_hole)
+		(attr through_hole exclude_from_bom dnp)
 		(fp_text user "${REFERENCE}"
 			(at 0 2.5 0)
@@
 		(sheetname "BB6V")
 		(sheetfile "bb6v.kicad_sch")
-		(attr through_hole exclude_from_bom)
+		(attr through_hole exclude_from_bom dnp)
 		(fp_circle
 			(center 0 0)
@@
 		(at 45.5 23.75)
 		(property "Reference" "RF101"
-			(at 0 -3 360)
+			(at 0 -3 0)
 			(layer "F.SilkS")
 			(effects
@@
 		)
 		(property "Value" "73412-0110"
-			(at 0 5.4 360)
+			(at 0 5.4 0)
 			(layer "F.Fab")
 			(effects
@@
 		)
 		(property "Footprint" "easyeda2kicad:ANT-SMD_73412-0110"
-			(at 0 0 360)
+			(at 0 0 0)
 			(layer "F.Fab")
 			(hide yes)
@@
 		)
 		(property "Datasheet" "https://lcsc.com/product-detail/RF-Connectors-Coaxial-Connectors_MOLEX-73412-0110_C434806.html"
-			(at 0 0 360)
+			(at 0 0 0)
 			(layer "F.Fab")
 			(hide yes)
@@
 		)
 		(property "Description" ""
-			(at 0 0 360)
+			(at 0 0 0)
 			(layer "F.Fab")
 			(hide yes)
@@
 		)
 		(fp_text user "${REFERENCE}"
-			(at 0 0 360)
+			(at 0 0 0)
 			(layer "F.Fab")
 			(effects
@@
 		(tags "capacitor")
 		(property "Reference" "C101"
-			(at 0 1.5 360)
+			(at 0 1.5 0)
 			(layer "F.SilkS")
 			(effects
@@
 			)
 		)
-		(property "Value" "C"
-			(at 0 1.43 360)
+		(property "Value" "10uf"
+			(at 0 1.43 0)
 			(layer "F.Fab")
 			(effects
@@
 		)
 		(fp_text user "${REFERENCE}"
-			(at 0 0 360)
+			(at 0 0 0)
 			(layer "F.Fab")
 			(effects
@@
 		(sheetname "Root")
 		(sheetfile "BuckBoostTest.kicad_sch")
-		(attr through_hole)
+		(attr through_hole exclude_from_bom dnp)
 		(fp_text user "${REFERENCE}"
 			(at 0 2.5 0)
@@
 		(at 36.83 54.25)
 		(property "Reference" "U101"
-			(at 8.92 0.25 360)
+			(at 8.92 0.25 0)
 			(layer "F.SilkS")
 			(effects
@@
 		)
 		(property "Value" "MC7805CDTRKG"
-			(at 0 6.29 360)
+			(at 0 6.29 0)
 			(layer "F.Fab")
 			(effects
@@
 		)
 		(property "Footprint" "easyeda2kicad:TO-252-2_L6.6-W6.1-P4.58-LS9.9-TL"
-			(at 0 0 360)
+			(at 0 0 0)
 			(layer "F.Fab")
 			(hide yes)
@@
 		)
 		(property "Datasheet" "https://lcsc.com/product-detail/Linear-Voltage-Regulators_ON_MC7805CDTRKG_MC7805CDTRKG_C54285.html"
-			(at 0 0 360)
+			(at 0 0 0)
 			(layer "F.Fab")
 			(hide yes)
@@
 		)
 		(property "Description" ""
-			(at 0 0 360)
+			(at 0 0 0)
 			(layer "F.Fab")
 			(hide yes)
@@
 		)
 		(fp_text user "${REFERENCE}"
-			(at 0 0 360)
+			(at 0 0 0)
 			(layer "F.Fab")
 			(effects
@@
 		(hatch edge 0.5)
 		(priority 5)
-		(connect_pads
+		(connect_pads yes
 			(clearance 0.5)
 		)

Commit message: revisions
Parts:
- C104: value 10f -> 10uf
Changed lines of the file:
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@@
 			)
 		)
-		(property "Value" "10f"
+		(property "Value" "10uf"
 			(at 0 1.43 0)
 			(layer "F.Fab")

Commit message: reannotate
Parts:
- renumbered C107 to C101, C106 to C102, C102 to C106, C101 to C107, RF103 to RF102, RF102 to RF103
Changed lines of the file:
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@@
 	(net 10 "Net-(RF104-SIG)")
 	(net 11 "Net-(U102-BYP)")
-	(net 12 "Net-(RF103-SIG)")
+	(net 12 "Net-(RF102-SIG)")
 	(net 13 "unconnected-(USB101-D--Pad2)")
 	(net 14 "unconnected-(USB101-D+-Pad3)")
@@
 		(layer "F.Cu")
 		(at 23.75 58.25 90)
-		(property "Reference" "RF103"
+		(property "Reference" "RF102"
 			(at 3.5 -0.37 180)
 			(layer "F.SilkS")
@@
 			(size 1.6 1)
 			(layers "F.Cu" "F.Paste" "F.Mask")
-			(net 12 "Net-(RF103-SIG)")
+			(net 12 "Net-(RF102-SIG)")
 			(pinfunction "SIG")
 			(pintype "unspecified")
@@
 			(size 1.2 3)
 			(layers "F.Cu" "F.Paste" "F.Mask")
-			(net 12 "Net-(RF103-SIG)")
+			(net 12 "Net-(RF102-SIG)")
 			(pinfunction "VCC")
 			(pintype "input")
@@
 		(layer "F.Cu")
 		(at 75.25 24.15)
-		(property "Reference" "RF102"
+		(property "Reference" "RF103"
 			(at 0 -5.4 0)
 			(layer "F.SilkS")
@@
 		(descr "Capacitor SMD 0603 (1608 Metric), square (rectangular) end terminal, IPC_7351 nominal, (Body size source: IPC-SM-782 page 76, https://www.pcb-3d.com/wordpress/wp-content/uploads/ipc-sm-782a_amendment_1_and_2.pdf), generated with kicad-footprint-generator")
 		(tags "capacitor")
-		(property "Reference" "C106"
+		(property "Reference" "C102"
 			(at 0 -1.43 0)
 			(layer "F.SilkS")
@@
 			(layers "F.Cu" "F.Paste" "F.Mask")
 			(roundrect_rratio 0.25)
-			(net 12 "Net-(RF103-SIG)")
+			(net 12 "Net-(RF102-SIG)")
 			(pintype "passive")
 		)
@@
 		(descr "Capacitor SMD 0603 (1608 Metric), square (rectangular) end terminal, IPC_7351 nominal, (Body size source: IPC-SM-782 page 76, https://www.pcb-3d.com/wordpress/wp-content/uploads/ipc-sm-782a_amendment_1_and_2.pdf), generated with kicad-footprint-generator")
 		(tags "capacitor")
-		(property "Reference" "C107"
+		(property "Reference" "C101"
 			(at -3.775 0 0)
 			(layer "F.SilkS")
@@
 		(descr "Capacitor SMD 0603 (1608 Metric), square (rectangular) end terminal, IPC_7351 nominal, (Body size source: IPC-SM-782 page 76, https://www.pcb-3d.com/wordpress/wp-content/uploads/ipc-sm-782a_amendment_1_and_2.pdf), generated with kicad-footprint-generator")
 		(tags "capacitor")
-		(property "Reference" "C102"
+		(property "Reference" "C106"
 			(at -0.025 1.75 90)
 			(layer "F.SilkS")
@@
 		(descr "Capacitor SMD 0603 (1608 Metric), square (rectangular) end terminal, IPC_7351 nominal, (Body size source: IPC-SM-782 page 76, https://www.pcb-3d.com/wordpress/wp-content/uploads/ipc-sm-782a_amendment_1_and_2.pdf), generated with kicad-footprint-generator")
 		(tags "capacitor")
-		(property "Reference" "C101"
+		(property "Reference" "C107"
 			(at 0 1.5 0)
 			(layer "F.SilkS")
@@
 			(size 2.41 0.98)
 			(layers "F.Cu" "F.Paste" "F.Mask")
-			(net 12 "Net-(RF103-SIG)")
+			(net 12 "Net-(RF102-SIG)")
 			(pinfunction "Output")
 			(pintype "unspecified")
