File: esp8266-flexpower/LED_comparator.kicad_sch (KiCad schematic)
At the start: 17 parts, among them U5 LM339

Commit message: ready to fab
Connections:
- net Input: now reaches U5.10 (-), U5.4 (-), U5.6 (-), U5.8 (-)
Changed lines of the file:
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@@
+		)
+	)
+	(hierarchical_label "Input"
+		(shape input)
+		(at 57.15 30.48 90)
+		(fields_autoplaced yes)
+		(effects
+			(font
+				(size 1.27 1.27)
+			)
+			(justify left)
 		)
 	)
