File: esp8266-flexpower/pp3v16v.kicad_sch (KiCad schematic)
At the start: 17 parts, among them Q1 2N7002

Commit message: ready to fab
Parts:
- JP1: footprint Connector_PinHeader_1.00mm:PinHeader_1x02_P1.00mm_Vertical -> Jumper:SolderJumper-2_P1.3mm_Bridged_Pad1.0x1.5mm
Changed lines of the file:
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@@
 	(paper "A4")
-	(junction
-		(at 116.84 43.18)
-		(diameter 0)
-		(color 0 0 0 0)
-	)
 	(junction
 		(at 54.61 38.1)
@@
 	(wire
 		(pts
-			(xy 116.84 43.18) (xy 120.65 43.18)
+			(xy 114.3 43.18) (xy 120.65 43.18)
 		)
 		(stroke
@@
 	(wire
 		(pts
-			(xy 116.84 43.18) (xy 116.84 64.77)
-		)
-		(stroke
-			(width 0)
-			(type default)
-		)
-	)
-	(wire
-		(pts
 			(xy 46.99 35.56) (xy 68.58 35.56)
 		)
@@
 		(pts
 			(xy 54.61 38.1) (xy 86.36 38.1)
-		)
-		(stroke
-			(width 0)
-			(type default)
-		)
-	)
-	(wire
-		(pts
-			(xy 114.3 43.18) (xy 116.84 43.18)
 		)
 		(stroke
@@
 			)
 		)
-		(property "Footprint" "Connector_PinHeader_1.00mm:PinHeader_1x02_P1.00mm_Vertical"
+		(property "Footprint" "Jumper:SolderJumper-2_P1.3mm_Bridged_Pad1.0x1.5mm"
 			(at 212.09 46.99 0)
 			(effects
