File: esp8266-flexpower/usb_serial.kicad_sch (KiCad schematic)
At the start: 14 parts, among them Q2 MMBT3904, Q3 MMBT3904, U2 USBLC6-2SC6, U3 CH340C

Commit message: ready to fab
Parts:
- R14, R15: value 480 -> 470
Connections:
- no-connect marks 4 -> 5
Changed lines of the file:
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@@
+	)
+	(no_connect
+		(at 119.38 86.36)
 	)
 	(no_connect
@@
 			)
 		)
-		(property "Value" "480"
+		(property "Value" "470"
 			(at 153.67 80.01 90)
 			(effects
@@
 			)
 		)
-		(property "Value" "480"
+		(property "Value" "470"
 			(at 153.416 91.44 90)
 			(effects
