File: surprise/pp3v16v.kicad_sch (KiCad schematic)
At the start: 19 parts, among them Q201 2N7002

Commit message: WIP: Revision2
Parts:
- renumbered TP202 to TP201, TP201 to TP202
Changed lines of the file:
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@@
 		(dnp no)
 		(fields_autoplaced yes)
-		(property "Reference" "TP202"
+		(property "Reference" "TP201"
 			(at 30.48 41.4019 0)
 			(effects
@@
 			(project "surprise"
 				(path "/48ddfdd8-68fa-4e63-aa18-bc113cdf8cfa/542ec963-64f2-405e-acad-a2c979ff5c5c"
-					(reference "TP202")
-					(unit 1)
-				)
-				(path "/48ddfdd8-68fa-4e63-aa18-bc113cdf8cfa/9d4f2f75-9e0d-4ff0-a99e-11be111d4b2b"
-					(reference "TP502")
+					(reference "TP201")
+					(unit 1)
+				)
+				(path "/48ddfdd8-68fa-4e63-aa18-bc113cdf8cfa/9d4f2f75-9e0d-4ff0-a99e-11be111d4b2b"
+					(reference "TP501")
 					(unit 1)
 				)
@@
 		(dnp no)
 		(fields_autoplaced yes)
-		(property "Reference" "TP201"
+		(property "Reference" "TP202"
 			(at 118.11 57.9119 0)
 			(effects
@@
 			(project "surprise"
 				(path "/48ddfdd8-68fa-4e63-aa18-bc113cdf8cfa/542ec963-64f2-405e-acad-a2c979ff5c5c"
-					(reference "TP201")
-					(unit 1)
-				)
-				(path "/48ddfdd8-68fa-4e63-aa18-bc113cdf8cfa/9d4f2f75-9e0d-4ff0-a99e-11be111d4b2b"
-					(reference "TP501")
-					(unit 1)
-				)
+					(reference "TP202")
+					(unit 1)
+				)
+				(path "/48ddfdd8-68fa-4e63-aa18-bc113cdf8cfa/9d4f2f75-9e0d-4ff0-a99e-11be111d4b2b"
+					(reference "TP502")
+					(unit 1)
+				)
