File: surprise/usb-c.kicad_sch (KiCad schematic)
At the start: 4 parts, among them U701 USBLC6-2SC6

Commit message: Ready to fab
Parts:
- added R702, R703: 5.1k, Resistor_SMD:R_0603_1608Metric, symbol Device:R
Connections:
- net GND: now also R702.2, R703.2
- net at USBC701.A5 (CC1): now also R702.1
- net at USBC701.B5 (CC2): now also R703.1
- no-connect marks 4 -> 2
Other:
- moved on the sheet: C701, R701, U701, USBC701
