File: surprise/surprise.kicad_sch (KiCad schematic)
At the start: 23 parts, among them J101 PM254V-11-07-H85, J102 HB-PH3-25413PB2GOP, U101 SN74LVC32ADR, U102 LP5912-3.3DRV, U103 LIS2DHTR

Commit message: WIP: Revision2
Parts:
- added D102, D103: WS2812B-2020, LED_SMD:LED_WS2812B-2020_PLCC4_2.0x2.0mm, symbol LED:WS2812B-2020
- added J103: Conn_01x03, Connector_JST:JST_PH_B3B-PH-K_1x03_P2.00mm_Vertical, symbol Connector_Generic:Conn_01x03
- renumbered J102 to J101, J101 to J102, JP104 to JP101, JP103 to JP102, JP107 to JP103, JP106 to JP104, JP108 to JP106, R103 to R102, R102 to R103
Connections:
- net +5V: now also D102.4 (VDD), D103.4 (VDD), J103.2 (Pin_2); no longer D101.4 (VDD)
- net GND: now also D102.2 (VSS), D103.2 (VSS), J103.1 (Pin_1)
- net at D101.1 (DOUT): now also D102.3 (DIN)
- net battery/VOUT renamed sys_power
- net sys_power: now also D101.4 (VDD)
- new net: D103.1 (DOUT), J103.3 (Pin_3)
- new net: D102.1 (DOUT), D103.3 (DIN)
- no-connect marks 19 -> 18
Other:
- moved on the sheet: D101, J102

Commit message: Ready to fab
Other:
- added sheet i2c (i2c.kicad_sch)
Changed lines of the file:
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@@
 	)
 	(junction
+		(at 120.65 148.59)
+		(diameter 0)
+		(color 0 0 0 0)
+	)
+	(junction
 		(at 153.67 156.21)
 		(diameter 0)
@@
 		(color 0 0 0 0)
 	)
+	(junction
+		(at 118.11 151.13)
+		(diameter 0)
+		(color 0 0 0 0)
+	)
 	(no_connect
 		(at 156.21 191.77)
@@
 	(wire
 		(pts
+			(xy 74.93 153.67) (xy 80.01 153.67)
+		)
+		(stroke
+			(width 0)
+			(type default)
+		)
+	)
+	(wire
+		(pts
 			(xy 210.82 29.21) (xy 223.52 29.21)
 		)
@@
 	(wire
 		(pts
+			(xy 93.98 148.59) (xy 120.65 148.59)
+		)
+		(stroke
+			(width 0)
+			(type default)
+		)
+	)
+	(wire
+		(pts
 			(xy 20.32 39.37) (xy 17.78 39.37)
 		)
@@
 	(wire
 		(pts
+			(xy 105.41 153.67) (xy 105.41 151.13)
+		)
+		(stroke
+			(width 0)
+			(type default)
+		)
+	)
+	(wire
+		(pts
 			(xy 198.12 119.38) (xy 220.98 119.38)
 		)
@@
 	(wire
 		(pts
+			(xy 71.12 148.59) (xy 81.28 148.59)
+		)
+		(stroke
+			(width 0)
+			(type default)
+		)
+	)
+	(wire
+		(pts
 			(xy 148.59 194.31) (xy 148.59 195.58)
 		)
@@
 	(wire
 		(pts
+			(xy 93.98 153.67) (xy 105.41 153.67)
+		)
+		(stroke
+			(width 0)
+			(type default)
+		)
+	)
+	(wire
+		(pts
 			(xy 45.72 66.04) (xy 171.45 66.04)
 		)
@@
 	(wire
 		(pts
+			(xy 105.41 151.13) (xy 118.11 151.13)
+		)
+		(stroke
+			(width 0)
+			(type default)
+		)
+	)
+	(wire
+		(pts
 			(xy 234.95 76.2) (xy 234.95 80.01)
 		)
@@
 	(global_label "3v3"
 		(shape input)
+		(at 74.93 153.67 180)
+		(fields_autoplaced yes)
+		(effects
+			(font
+				(size 1.27 1.27)
+			)
+			(justify right)
+		)
+		(property "Intersheetrefs" "${INTERSHEET_REFS}"
+			(at 68.5582 153.67 0)
+			(effects
+				(font
+					(size 1.27 1.27)
+				)
+				(justify right)
+				(hide yes)
+			)
+		)
+	)
+	(global_label "3v3"
+		(shape input)
 		(at 234.95 76.2 180)
 		(fields_autoplaced yes)
@@
 	)
 	(symbol
+		(lib_id "power:+5V")
+		(at 71.12 148.59 90)
+		(unit 1)
+		(exclude_from_sim no)
+		(in_bom yes)
+		(on_board yes)
+		(dnp no)
+		(fields_autoplaced yes)
+		(property "Reference" "#PWR0116"
+			(at 74.93 148.59 0)
+			(effects
+				(font
+					(size 1.27 1.27)
+				)
+				(hide yes)
+			)
+		)
+		(property "Value" "+5V"
+			(at 67.31 148.5899 90)
+			(effects
+				(font
+					(size 1.27 1.27)
+				)
+				(justify left)
+			)
+		)
+		(property "Footprint" ""
+			(at 71.12 148.59 0)
+			(effects
+				(font
+					(size 1.27 1.27)
+				)
+				(hide yes)
+			)
+		)
+		(property "Datasheet" ""
+			(at 71.12 148.59 0)
+			(effects
+				(font
+					(size 1.27 1.27)
+				)
+				(hide yes)
+			)
+		)
+		(property "Description" "Power symbol creates a global label with name \"+5V\""
+			(at 71.12 148.59 0)
+			(effects
+				(font
+					(size 1.27 1.27)
+				)
+				(hide yes)
+			)
+		)
+		(pin "1"
+		)
+		(instances
+			(project "surprise"
+				(path "/48ddfdd8-68fa-4e63-aa18-bc113cdf8cfa"
+					(reference "#PWR0116")
+					(unit 1)
+				)
+			)
+		)
+	)
+	(symbol
 		(lib_id "LED:WS2812B-2020")
 		(at 229.87 138.43 0)
@@
 				)
 			)
+		)
+	)
+	(sheet
+		(at 80.01 145.415)
+		(size 15.24 12.7)
+		(fields_autoplaced yes)
+		(stroke
+			(width 0.1524)
+			(type solid)
+		)
+		(fill
+			(color 0 0 0 0.0000)
+		)
+		(property "Sheetname" "i2c"
+			(at 80.01 144.7034 0)
+			(effects
+				(font
+					(size 1.27 1.27)
+				)
+				(justify left bottom)
+			)
+		)
+		(property "Sheetfile" "i2c.kicad_sch"
+			(at 80.01 158.6996 0)
+			(effects
+				(font
+					(size 1.27 1.27)
+				)
+				(justify left top)
+			)
+		)
+		(pin "SDA" input
+			(at 95.25 148.59 0)
+			(effects
+				(font
+					(size 1.27 1.27)
+				)
+				(justify right)
+			)
+		)
+		(pin "VCC" input
+			(at 80.01 148.59 180)
+			(effects
+				(font
+					(size 1.27 1.27)
+				)
+				(justify left)
+			)
+		)
+		(pin "3V3" input
+			(at 80.01 153.67 180)
+			(effects
+				(font
+					(size 1.27 1.27)
+				)
+				(justify left)
+			)
+		)
+		(pin "SCL" input
+			(at 95.25 153.67 0)
+			(effects
+				(font
+					(size 1.27 1.27)
+				)
+				(justify right)
+			)
+		)
+		(instances
+			(project "surprise"
+				(path "/48ddfdd8-68fa-4e63-aa18-bc113cdf8cfa"
+					(page "13")
+				)
+			)

Commit message: add part numbers
Parts:
- J103: LCSC Part (none) -> C131339
Changed lines of the file:
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@@
+			)
+		)
+		(property "LCSC Part" "C131339"
+			(at 262.89 146.05 90)
+			(effects
+				(font
+					(size 1.27 1.27)
+				)
+				(hide yes)
 			)
 		)

Commit message: add resistor size reference guide
Other:
- added sheet components (components.kicad_sch)
Changed lines of the file:
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@@
+	)
+	(sheet
+		(at 63.5 26.67)
+		(size 16.51 13.97)
+		(fields_autoplaced yes)
+		(stroke
+			(width 0.1524)
+			(type solid)
+		)
+		(fill
+			(color 0 0 0 0.0000)
+		)
+		(property "Sheetname" "components"
+			(at 63.5 25.9584 0)
+			(effects
+				(font
+					(size 1.27 1.27)
+				)
+				(justify left bottom)
+			)
+		)
+		(property "Sheetfile" "components.kicad_sch"
+			(at 63.5 41.2246 0)
+			(effects
+				(font
+					(size 1.27 1.27)
+				)
+				(justify left top)
+			)
+		)
+		(instances
+			(project "surprise"
+				(path "/48ddfdd8-68fa-4e63-aa18-bc113cdf8cfa"
+					(page "14")
+				)
+			)
+		)
 	)
 	(sheet
