File: usbserial/usbserial.kicad_sch (KiCad schematic)
At the start: 0 parts

Commit message: WIP: usbserial
Parts:
- added J101: Conn_01x06, Connector_PinHeader_2.54mm:PinHeader_1x06_P2.54mm_Vertical, symbol Connector_Generic:Conn_01x06
Connections:
- net usb_serial/BOOT: now also J101.5 (Pin_5)
- net usb_serial/RST: now also J101.6 (Pin_6)
- net usb_serial/RXD: now also J101.4 (Pin_4)
- net usb_serial/TXD: now also J101.3 (Pin_3)
- net usb_serial/VUSB: now also J101.1 (Pin_1)
- new net GND: J101.2 (Pin_2)

Commit message: work on usbserial
Parts:
- added C101, C102, C103: 1uF, Capacitor_SMD:C_0603_1608Metric, symbol Device:C
- added C104: 10nF, Capacitor_SMD:C_0603_1608Metric, symbol Device:C
- added J102: Conn_02x02_Counter_Clockwise, Connector_PinHeader_2.54mm:PinHeader_2x02_P2.54mm_Vertical, symbol Connector_Generic:Conn_02x02_Counter_Clockwise
- added R101: 10k, Resistor_SMD:R_0603_1608Metric, symbol Device:R
- added U101: TPS73733DCQ_C5220270, easyeda2kicad:SOT-223-6_L6.5-W3.5-P1.27-LS7.0-BR, symbol easyeda2kicad:TPS73733DCQ_C5220270
Connections:
- net GND: now also C101.2, C102.2, C103.2, C104.2, U101.3 (GND), U101.6 (GND)
- net usb_serial/VUSB: now also C101.1, J102.1 (Pin_1), R101.1, U101.1 (IN); no longer J101.1 (Pin_1)
- new net: C104.1, U101.4 (NR/FB)
- new net: R101.2, U101.5 (EN)
- new net 3v3: C102.1, C103.1, J102.2 (Pin_2), U101.2 (OUT)
- new net PWR: J101.1 (Pin_1), J102.3 (Pin_3), J102.4 (Pin_4)
Other:
- moved on the sheet: J101

Commit message: usbserial v2
Parts:
- J102: LCSC Part (none) -> C18078211
Changed lines of the file:
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@@
+			)
+		)
+		(property "LCSC Part" "C18078211"
+			(at 166.37 58.42 0)
+			(effects
+				(font
+					(size 1.27 1.27)
+				)
+				(hide yes)
 			)
 		)
