File: usbserial/usbserial.kicad_sch (KiCad schematic)
At the start: 8 parts, among them J101 Conn_01x06, J102 Conn_02x02_Counter_Clockwise, U101 TPS73733DCQ_C5220270

Commit message: usbserial: run CH340C from 3.3 V so target-facing signals are 3.3 V
The CH340C was powered from VUSB, so TXD, DTR and RTS swung to ~5 V
into ESP32 pins that are not 5 V tolerant. Power it from the TPS73733
3v3 rail instead, using the chip's 3.3 V configuration (V3 tied to VCC).

Schematic:
- U402 VCC and V3 on 3v3; C404 decouples the node.
- C403 (the 100 nF next to pin 16) moves from VUSB to 3v3 with it.
- New 3v3 sheet pin on usb_serial, fed from the root 3v3 rail.

PCB:
- Pin 16: F.Cu to C403, via + B.Cu to J102 pin 2.
- Pin 4: via under the body, B.Cu inside the TXD/RXD channel, via +
  F.Cu stub to J102 pin 2. Routed so no ground pour is enclosed.
- Direct trace from C402 to its VUSB via, since C403 left that pour.
- Zones refilled. Saving through the KiCad 9 API upgraded the file
  format from KiCad 8.

ERC is one error better than before; DRC matches the previous 28
violations with no unconnected pads and clean schematic parity.
production/ outputs are not regenerated.

Co-Authored-By: Claude Opus 5.5 <noreply@anthropic.com>
Other:
- sheet usb_serial ports: added 3v3; removed none
Changed lines of the file:
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@@
+	)
+	(label "3v3"
+		(at 81.28 97.79 0)
+		(effects
+			(font
+				(size 1.27 1.27)
+			)
+			(justify left bottom)
+		)
+	)
+	(wire
+		(pts
+			(xy 73.66 97.79) (xy 81.28 97.79)
+		)
+		(stroke
+			(width 0)
+			(type default)
+		)
 	)
 	(label "3v3"
@@
 			)
 		)
+		(pin "3v3" input
+			(at 73.66 97.79 0)
+			(effects
+				(font
+					(size 1.27 1.27)
+				)
+				(justify right)
+			)
+		)

Commit message: usbserial v0.2: TX/RX LEDs, design-review fixes, JLCPCB outputs
Add TX/RX activity LEDs and fix the issues found in a design review,
then regenerate the JLCPCB production files and document the board.

TX/RX LEDs (JLCPCB basic parts):
- D401/D402 red 0603 LED (C2286) + R406/R407 1k (C21190), 3v3 -> R ->
  LED -> line, so each lights while its UART line is low (~1.4 mA).
- TX taps the CH340C side of R402 (new net CH340_TXD); RX taps the
  connector side of R403 so the LED current does not drop across R403.
- Placed lower-left beside the CH340C with a TX/RX silk legend; 3v3 is
  brought in on B.Cu from a via on the C403 trace.

Review fixes:
- USB-C shell tabs were floating: tie them to GND.
- USB-C locating pegs were PTH with a zero annular ring: make them NPTH.
- R402/R403 487 -> 470 ohm (basic part).
- U101 GND pin 3 starved thermal: solid connection plus a direct trace
  to C102 ground.
- No-connect flags on SBU1/SBU2/R232, PWR_FLAG on GND, remove two
  dangling wire stubs, fill in title blocks.
- Silk text line width 0.10 -> 0.15 mm; clip connector silk to the
  board edge.
- LCSC Part / MPN / Manufacturer on every part.

Fabrication:
- production/ was generated before the CH340C moved to 3.3 V; regenerate
  Gerbers, drills, IPC-D-356, BOM and CPL from this board.
- The CPL used to rotate U101 by 180 degrees: Fabrication Toolkit's
  ^SOT-223 rule also matches the easyeda2kicad footprint, which is
  already in LCSC orientation. Use 180 (no correction) and add
  FT Rotation Offset = -180 so the Toolkit reproduces it.

ERC errors 9 -> 0, DRC errors 3 -> 0, no unconnected items, schematic
parity clean (KiCad 9.0.9). Datasheet PDFs could not be fetched from
this environment; the README lists sources and the sync command.

Co-Authored-By: Claude Opus 5.5 <noreply@anthropic.com>
Claude-Session: https://claude.ai/code/session_01GBv2vfRdNQ19uomtXMey2j
Parts:
- C101, C102, C103: LCSC Part (none) -> C15849; MPN (none) -> CL10A105KB8NNNC; Manufacturer (none) -> Samsung Electro-Mechanics
- C104: LCSC Part (none) -> C57112; MPN (none) -> CL10B103KB8NNNC; Manufacturer (none) -> Samsung Electro-Mechanics
- R101: LCSC Part (none) -> C25804; MPN (none) -> 0603WAF1002T5E; Manufacturer (none) -> UNI-ROYAL(Uniroyal Elec)
- U101: FT Rotation Offset (none) -> -180; MPN (none) -> TPS73733DCQR; Manufacturer (none) -> Texas Instruments
Other:
- title: (none) -> USB Serial Flasher
Changed lines of the file:
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@@
 	(generator_version "8.0")
 	(paper "A4")
+	(title_block
+		(title "USB Serial Flasher")
+		(date "2026-11-01")
+		(rev "0.2")
+		(comment 1 "Power: TPS73733 3.3 V LDO, target supply jumper")
+	)
 	(junction
 		(at 121.92 76.2)
@@
 			)
 		)
-		(property "Datasheet" ""
+		(property "Datasheet" "https://www.ti.com/lit/ds/symlink/tps737.pdf"
 			(at 121.92 66.04 0)
 			(effects
@@
 		(property "LCSC Part" "C5220270"
 			(at 121.92 81.28 0)
+			(effects
+				(font
+					(size 1.27 1.27)
+				)
+				(hide yes)
+			)
+		)
+		(property "MPN" "TPS73733DCQR"
+			(at 121.92 66.04 0)
+			(effects
+				(font
+					(size 1.27 1.27)
+				)
+				(hide yes)
+			)
+		)
+		(property "Manufacturer" "Texas Instruments"
+			(at 121.92 66.04 0)
+			(effects
+				(font
+					(size 1.27 1.27)
+				)
+				(hide yes)
+			)
+		)
+		(property "FT Rotation Offset" "-180"
+			(at 121.92 66.04 0)
 			(effects
 				(font
@@
 			)
 		)
+		(property "LCSC Part" "C15849"
+			(at 148.59 64.77 0)
+			(effects
+				(font
+					(size 1.27 1.27)
+				)
+				(hide yes)
+			)
+		)
+		(property "MPN" "CL10A105KB8NNNC"
+			(at 148.59 64.77 0)
+			(effects
+				(font
+					(size 1.27 1.27)
+				)
+				(hide yes)
+			)
+		)
+		(property "Manufacturer" "Samsung Electro-Mechanics"
+			(at 148.59 64.77 0)
+			(effects
+				(font
+					(size 1.27 1.27)
+				)
+				(hide yes)
+			)
+		)
 		(pin "1"
 		)
@@
 			)
 		)
+		(property "LCSC Part" "C25804"
+			(at 110.49 54.61 0)
+			(effects
+				(font
+					(size 1.27 1.27)
+				)
+				(hide yes)
+			)
+		)
+		(property "MPN" "0603WAF1002T5E"
+			(at 110.49 54.61 0)
+			(effects
+				(font
+					(size 1.27 1.27)
+				)
+				(hide yes)
+			)
+		)
+		(property "Manufacturer" "UNI-ROYAL(Uniroyal Elec)"
+			(at 110.49 54.61 0)
+			(effects
+				(font
+					(size 1.27 1.27)
+				)
+				(hide yes)
+			)
+		)
 		(pin "2"
 		)
@@
 			)
 		)
+		(property "LCSC Part" "C15849"
+			(at 95.25 64.77 0)
+			(effects
+				(font
+					(size 1.27 1.27)
+				)
+				(hide yes)
+			)
+		)
+		(property "MPN" "CL10A105KB8NNNC"
+			(at 95.25 64.77 0)
+			(effects
+				(font
+					(size 1.27 1.27)
+				)
+				(hide yes)
+			)
+		)
+		(property "Manufacturer" "Samsung Electro-Mechanics"
+			(at 95.25 64.77 0)
+			(effects
+				(font
+					(size 1.27 1.27)
+				)
+				(hide yes)
+			)
+		)
 		(pin "1"
 		)
@@
 			)
 		)
+		(property "LCSC Part" "C15849"
+			(at 135.89 64.77 0)
+			(effects
+				(font
+					(size 1.27 1.27)
+				)
+				(hide yes)
+			)
+		)
+		(property "MPN" "CL10A105KB8NNNC"
+			(at 135.89 64.77 0)
+			(effects
+				(font
+					(size 1.27 1.27)
+				)
+				(hide yes)
+			)
+		)
+		(property "Manufacturer" "Samsung Electro-Mechanics"
+			(at 135.89 64.77 0)
+			(effects
+				(font
+					(size 1.27 1.27)
+				)
+				(hide yes)
+			)
+		)
 		(pin "1"
 		)
@@
 			)
 		)
+		(property "LCSC Part" "C57112"
+			(at 105.41 71.12 0)
+			(effects
+				(font
+					(size 1.27 1.27)
+				)
+				(hide yes)
+			)
+		)
+		(property "MPN" "CL10B103KB8NNNC"
+			(at 105.41 71.12 0)
+			(effects
+				(font
+					(size 1.27 1.27)
+				)
+				(hide yes)
+			)
+		)
+		(property "Manufacturer" "Samsung Electro-Mechanics"
+			(at 105.41 71.12 0)
+			(effects
+				(font
+					(size 1.27 1.27)
+				)
+				(hide yes)
+			)
+		)
 		(pin "1"
 		)
@@
 				)
 			)
+		)
+	)
+	(symbol
+		(lib_id "power:PWR_FLAG")
+		(at 95.25 76.2 180)
+		(unit 1)
+		(exclude_from_sim no)
+		(in_bom yes)
+		(on_board yes)
+		(dnp no)
+		(property "Reference" "#FLG0101"
+			(at 95.25 78.105 0)
+			(effects
+				(font
+					(size 1.27 1.27)
+				)
+				(hide yes)
+			)
+		)
+		(property "Value" "PWR_FLAG"
+			(at 95.25 80.01 0)
+			(effects
+				(font
+					(size 1.27 1.27)
+				)
+			)
+		)
+		(property "Footprint" ""
+			(at 95.25 76.2 0)
+			(effects
+				(font
+					(size 1.27 1.27)
+				)
+				(hide yes)
+			)
+		)
+		(property "Datasheet" "~"
+			(at 95.25 76.2 0)
+			(effects
+				(font
+					(size 1.27 1.27)
+				)
+				(hide yes)
+			)
+		)
+		(property "Description" "Special symbol for telling ERC where power comes from"
+			(at 95.25 76.2 0)
+			(effects
+				(font
+					(size 1.27 1.27)
+				)
+				(hide yes)
+			)
+		)
+		(pin "1"
+		)
+		(instances
+			(project ""
+				(path "/48ddfdd8-68fa-4e63-aa18-bc113cdf8cfa"
+					(reference "#FLG0101")
+					(unit 1)
+				)
+			)
