File: usbserial/usbserial.kicad_pcb (KiCad board)
At the start: 4 copper layers, 40 x 36.8 mm, 23 parts, among them J101 Conn_01x06, J102 Conn_02x02_Counter_Clockwise, Q401 MMBT3904, Q402 MMBT3904, U101 TPS73733DCQ_C5220270, U401 USBLC6-2SC6, U402 CH340C

Commit message: usbserial: run CH340C from 3.3 V so target-facing signals are 3.3 V
The CH340C was powered from VUSB, so TXD, DTR and RTS swung to ~5 V
into ESP32 pins that are not 5 V tolerant. Power it from the TPS73733
3v3 rail instead, using the chip's 3.3 V configuration (V3 tied to VCC).

Schematic:
- U402 VCC and V3 on 3v3; C404 decouples the node.
- C403 (the 100 nF next to pin 16) moves from VUSB to 3v3 with it.
- New 3v3 sheet pin on usb_serial, fed from the root 3v3 rail.

PCB:
- Pin 16: F.Cu to C403, via + B.Cu to J102 pin 2.
- Pin 4: via under the body, B.Cu inside the TXD/RXD channel, via +
  F.Cu stub to J102 pin 2. Routed so no ground pour is enclosed.
- Direct trace from C402 to its VUSB via, since C403 left that pour.
- Zones refilled. Saving through the KiCad 9 API upgraded the file
  format from KiCad 8.

ERC is one error better than before; DRC matches the previous 28
violations with no unconnected pads and clean schematic parity.
production/ outputs are not regenerated.

Co-Authored-By: Claude Opus 5.5 <noreply@anthropic.com>
Connections:
- C403 pad 1: /usb_serial/VUSB -> /3v3
- C404 pad 2: Net-(U402-V3) -> /3v3
- U402 pad 16: /usb_serial/VUSB -> /3v3
- U402 pad 4: Net-(U402-V3) -> /3v3
Routing:
- net /3v3: track 0.00 -> 51.7 mm, vias 0 -> 3
- net Net-(U402-V3): track 2.21 -> 0.00 mm
- net /usb_serial/VUSB: track 10.9 -> 12.3 mm

Commit message: usbserial v0.2: TX/RX LEDs, design-review fixes, JLCPCB outputs
Add TX/RX activity LEDs and fix the issues found in a design review,
then regenerate the JLCPCB production files and document the board.

TX/RX LEDs (JLCPCB basic parts):
- D401/D402 red 0603 LED (C2286) + R406/R407 1k (C21190), 3v3 -> R ->
  LED -> line, so each lights while its UART line is low (~1.4 mA).
- TX taps the CH340C side of R402 (new net CH340_TXD); RX taps the
  connector side of R403 so the LED current does not drop across R403.
- Placed lower-left beside the CH340C with a TX/RX silk legend; 3v3 is
  brought in on B.Cu from a via on the C403 trace.

Review fixes:
- USB-C shell tabs were floating: tie them to GND.
- USB-C locating pegs were PTH with a zero annular ring: make them NPTH.
- R402/R403 487 -> 470 ohm (basic part).
- U101 GND pin 3 starved thermal: solid connection plus a direct trace
  to C102 ground.
- No-connect flags on SBU1/SBU2/R232, PWR_FLAG on GND, remove two
  dangling wire stubs, fill in title blocks.
- Silk text line width 0.10 -> 0.15 mm; clip connector silk to the
  board edge.
- LCSC Part / MPN / Manufacturer on every part.

Fabrication:
- production/ was generated before the CH340C moved to 3.3 V; regenerate
  Gerbers, drills, IPC-D-356, BOM and CPL from this board.
- The CPL used to rotate U101 by 180 degrees: Fabrication Toolkit's
  ^SOT-223 rule also matches the easyeda2kicad footprint, which is
  already in LCSC orientation. Use 180 (no correction) and add
  FT Rotation Offset = -180 so the Toolkit reproduces it.

ERC errors 9 -> 0, DRC errors 3 -> 0, no unconnected items, schematic
parity clean (KiCad 9.0.9). Datasheet PDFs could not be fetched from
this environment; the README lists sources and the sync command.

Co-Authored-By: Claude Opus 5.5 <noreply@anthropic.com>
Claude-Session: https://claude.ai/code/session_01GBv2vfRdNQ19uomtXMey2j
Parts:
- added D401: LED, LED_SMD:LED_0603_1608Metric, F.Cu at (26.6, 44.3)
- added D402: LED, LED_SMD:LED_0603_1608Metric, F.Cu at (28.6, 44.3)
- added R406: 1k, Resistor_SMD:R_0603_1608Metric, F.Cu at (26.6, 47.4)
- added R407: 1k, Resistor_SMD:R_0603_1608Metric, F.Cu at (28.6, 47.4)
- C401, C403, C404: value 100nf -> 100nF
- C402: value 10uf -> 10uF
- R402, R403: value 487 -> 470
Connections:
- net Net-(U402-TXD) renamed /usb_serial/CH340_TXD
- USBC201 pad 0: unconnected-(USBC201-SH-Pad0) -> GND
- USBC201 pad 1: unconnected-(USBC201-SH-Pad1) -> GND
- USBC201 pad 2: unconnected-(USBC201-SH-Pad2) -> GND
- USBC201 pad 3: unconnected-(USBC201-SH-Pad3) -> GND
Routing:
- net /3v3: track 51.7 -> 69.1 mm, vias 3 -> 5
- net /usb_serial/CH340_TXD: track 2.42 -> 10.6 mm
- net /usb_serial/RXD: track 34.8 -> 39.2 mm
- net GND: track 9.70 -> 12.3 mm
- net Net-(D402-A): track 0.00 -> 1.49 mm
- net Net-(D401-A): track 0.00 -> 1.49 mm
Other:
- board text added: "RX"
- board text added: "TX"
- board text added: "USB-Serial v0.2"
- board text removed: "USB-Serial v0.1"
