File: leds/3v3.kicad_sch (KiCad schematic)
At the start: 6 parts, among them U701 TPS73733DCQ_C5220270

Commit message: first draft
Parts:
- renumbered C701 to C24, C702 to C25, C703 to C26, C704 to C27, R701 to R23, U701 to U7
Changed lines of the file:
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@@
 		(dnp no)
 		(fields_autoplaced yes)
-		(property "Reference" "C702"
+		(property "Reference" "C25"
 			(at 88.9 77.4699 0)
 			(effects
@@
 			(project "espamp"
 				(path "/48ddfdd8-68fa-4e63-aa18-bc113cdf8cfa/ff982210-6c86-422a-a66b-20bff67bd030"
-					(reference "C702")
+					(reference "C25")
 					(unit 1)
 				)
@@
 		(dnp no)
 		(fields_autoplaced yes)
-		(property "Reference" "R701"
+		(property "Reference" "R23"
 			(at 90.17 55.88 90)
 			(effects
@@
 			(project "espamp"
 				(path "/48ddfdd8-68fa-4e63-aa18-bc113cdf8cfa/ff982210-6c86-422a-a66b-20bff67bd030"
-					(reference "R701")
+					(reference "R23")
 					(unit 1)
 				)
@@
 		(dnp no)
 		(fields_autoplaced yes)
-		(property "Reference" "C703"
+		(property "Reference" "C26"
 			(at 119.38 71.1199 0)
 			(effects
@@
 			(project "espamp"
 				(path "/48ddfdd8-68fa-4e63-aa18-bc113cdf8cfa/ff982210-6c86-422a-a66b-20bff67bd030"
-					(reference "C703")
+					(reference "C26")
 					(unit 1)
 				)
@@
 		(on_board yes)
 		(dnp no)
-		(property "Reference" "U701"
+		(property "Reference" "U7"
 			(at 108.712 64.262 0)
 			(effects
@@
 			(project "espamp"
 				(path "/48ddfdd8-68fa-4e63-aa18-bc113cdf8cfa/ff982210-6c86-422a-a66b-20bff67bd030"
-					(reference "U701")
+					(reference "U7")
 					(unit 1)
 				)
@@
 		(dnp no)
 		(fields_autoplaced yes)
-		(property "Reference" "#PWR0601"
+		(property "Reference" "#PWR029"
 			(at 110.49 90.17 0)
 			(effects
@@
 			(project ""
 				(path "/48ddfdd8-68fa-4e63-aa18-bc113cdf8cfa/ff982210-6c86-422a-a66b-20bff67bd030"
-					(reference "#PWR0601")
+					(reference "#PWR029")
 					(unit 1)
 				)
@@
 		(dnp no)
 		(fields_autoplaced yes)
-		(property "Reference" "C704"
+		(property "Reference" "C27"
 			(at 132.08 71.1199 0)
 			(effects
@@
 			(project "espamp"
 				(path "/48ddfdd8-68fa-4e63-aa18-bc113cdf8cfa/ff982210-6c86-422a-a66b-20bff67bd030"
-					(reference "C704")
+					(reference "C27")
 					(unit 1)
 				)
@@
 		(dnp no)
 		(fields_autoplaced yes)
-		(property "Reference" "C701"
+		(property "Reference" "C24"
 			(at 78.74 71.1199 0)
 			(effects
@@
 			(project "espamp"
 				(path "/48ddfdd8-68fa-4e63-aa18-bc113cdf8cfa/ff982210-6c86-422a-a66b-20bff67bd030"
-					(reference "C701")
-					(unit 1)
-				)
+					(reference "C24")
+					(unit 1)
+				)
