File: leds/buckconverter.kicad_sch (KiCad schematic)
At the start: 12 parts, among them U401 TPS54202DDC, U402 CYA1040-15UH

Commit message: first draft
Parts:
- renumbered C401 to C18, C402 to C19, C403 to C20, C404 to C21, C405 to C22, C406 to C23, R401 to R18, R402 to R19, R403 to R20, TP401 to TP4, U401 to U5, U402 to U6
Changed lines of the file:
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@@
 		(dnp no)
 		(fields_autoplaced yes)
-		(property "Reference" "#PWR0404"
+		(property "Reference" "#PWR027"
 			(at 142.24 73.66 0)
 			(effects
@@
 			(project ""
 				(path "/48ddfdd8-68fa-4e63-aa18-bc113cdf8cfa/aa9739d0-05d8-4c74-a4fd-846c263eed0b"
-					(reference "#PWR0404")
+					(reference "#PWR027")
 					(unit 1)
 				)
@@
 		(dnp no)
 		(fields_autoplaced yes)
-		(property "Reference" "#PWR0401"
+		(property "Reference" "#PWR024"
 			(at 38.1 49.53 0)
 			(effects
@@
 			(project ""
 				(path "/48ddfdd8-68fa-4e63-aa18-bc113cdf8cfa/aa9739d0-05d8-4c74-a4fd-846c263eed0b"
-					(reference "#PWR0401")
+					(reference "#PWR024")
 					(unit 1)
 				)
@@
 		(dnp no)
 		(fields_autoplaced yes)
-		(property "Reference" "R402"
+		(property "Reference" "R19"
 			(at 144.78 45.7199 0)
 			(effects
@@
 			(project ""
 				(path "/48ddfdd8-68fa-4e63-aa18-bc113cdf8cfa/aa9739d0-05d8-4c74-a4fd-846c263eed0b"
-					(reference "R402")
+					(reference "R19")
 					(unit 1)
 				)
@@
 		(dnp no)
 		(fields_autoplaced yes)
-		(property "Reference" "C406"
+		(property "Reference" "C23"
 			(at 134.62 45.7199 0)
 			(effects
@@
 			(project ""
 				(path "/48ddfdd8-68fa-4e63-aa18-bc113cdf8cfa/aa9739d0-05d8-4c74-a4fd-846c263eed0b"
-					(reference "C406")
+					(reference "C23")
 					(unit 1)
 				)
@@
 		(dnp no)
 		(fields_autoplaced yes)
-		(property "Reference" "C402"
+		(property "Reference" "C19"
 			(at 49.53 27.9399 0)
 			(effects
@@
 			(project ""
 				(path "/48ddfdd8-68fa-4e63-aa18-bc113cdf8cfa/aa9739d0-05d8-4c74-a4fd-846c263eed0b"
-					(reference "C402")
+					(reference "C19")
 					(unit 1)
 				)
@@
 		(dnp no)
 		(fields_autoplaced yes)
-		(property "Reference" "R401"
+		(property "Reference" "R18"
 			(at 144.78 34.2899 0)
 			(effects
@@
 			(project ""
 				(path "/48ddfdd8-68fa-4e63-aa18-bc113cdf8cfa/aa9739d0-05d8-4c74-a4fd-846c263eed0b"
-					(reference "R401")
+					(reference "R18")
 					(unit 1)
 				)
@@
 		(dnp no)
 		(fields_autoplaced yes)
-		(property "Reference" "U401"
+		(property "Reference" "U5"
 			(at 73.66 20.32 0)
 			(effects
@@
 			(project ""
 				(path "/48ddfdd8-68fa-4e63-aa18-bc113cdf8cfa/aa9739d0-05d8-4c74-a4fd-846c263eed0b"
-					(reference "U401")
+					(reference "U5")
 					(unit 1)
 				)
@@
 		(dnp no)
 		(fields_autoplaced yes)
-		(property "Reference" "C401"
+		(property "Reference" "C18"
 			(at 38.1 27.9399 0)
 			(effects
@@
 			(project ""
 				(path "/48ddfdd8-68fa-4e63-aa18-bc113cdf8cfa/aa9739d0-05d8-4c74-a4fd-846c263eed0b"
-					(reference "C401")
+					(reference "C18")
 					(unit 1)
 				)
@@
 		(dnp no)
 		(fields_autoplaced yes)
-		(property "Reference" "#PWR0403"
+		(property "Reference" "#PWR026"
 			(at 115.57 52.07 0)
 			(effects
@@
 			(project ""
 				(path "/48ddfdd8-68fa-4e63-aa18-bc113cdf8cfa/aa9739d0-05d8-4c74-a4fd-846c263eed0b"
-					(reference "#PWR0403")
+					(reference "#PWR026")
 					(unit 1)
 				)
@@
 		(dnp no)
 		(fields_autoplaced yes)
-		(property "Reference" "C405"
+		(property "Reference" "C22"
 			(at 124.46 34.6709 0)
 			(effects
@@
 			(project ""
 				(path "/48ddfdd8-68fa-4e63-aa18-bc113cdf8cfa/aa9739d0-05d8-4c74-a4fd-846c263eed0b"
-					(reference "C405")
+					(reference "C22")
 					(unit 1)
 				)
@@
 		(dnp no)
 		(fields_autoplaced yes)
-		(property "Reference" "U402"
+		(property "Reference" "U6"
 			(at 104.14 21.59 0)
 			(effects
@@
 			(project ""
 				(path "/48ddfdd8-68fa-4e63-aa18-bc113cdf8cfa/aa9739d0-05d8-4c74-a4fd-846c263eed0b"
-					(reference "U402")
+					(reference "U6")
 					(unit 1)
 				)
@@
 		(dnp no)
 		(fields_autoplaced yes)
-		(property "Reference" "TP401"
+		(property "Reference" "TP4"
 			(at 134.62 23.622 0)
 			(effects
@@
 			(project "espamp"
 				(path "/48ddfdd8-68fa-4e63-aa18-bc113cdf8cfa/aa9739d0-05d8-4c74-a4fd-846c263eed0b"
-					(reference "TP401")
+					(reference "TP4")
 					(unit 1)
 				)
@@
 		(dnp no)
 		(fields_autoplaced yes)
-		(property "Reference" "C403"
+		(property "Reference" "C20"
 			(at 93.98 20.32 90)
 			(effects
@@
 			(project ""
 				(path "/48ddfdd8-68fa-4e63-aa18-bc113cdf8cfa/aa9739d0-05d8-4c74-a4fd-846c263eed0b"
-					(reference "C403")
+					(reference "C20")
 					(unit 1)
 				)
@@
 		(dnp no)
 		(fields_autoplaced yes)
-		(property "Reference" "C404"
+		(property "Reference" "C21"
 			(at 113.03 34.6709 0)
 			(effects
@@
 			(project ""
 				(path "/48ddfdd8-68fa-4e63-aa18-bc113cdf8cfa/aa9739d0-05d8-4c74-a4fd-846c263eed0b"
-					(reference "C404")
+					(reference "C21")
 					(unit 1)
 				)
@@
 		(dnp no)
 		(fields_autoplaced yes)
-		(property "Reference" "R403"
+		(property "Reference" "R20"
 			(at 144.78 57.1499 0)
 			(effects
@@
 			(project ""
 				(path "/48ddfdd8-68fa-4e63-aa18-bc113cdf8cfa/aa9739d0-05d8-4c74-a4fd-846c263eed0b"
-					(reference "R403")
+					(reference "R20")
 					(unit 1)
 				)
@@
 		(dnp no)
 		(fields_autoplaced yes)
-		(property "Reference" "#PWR0402"
+		(property "Reference" "#PWR025"
 			(at 73.66 49.53 0)
 			(effects
@@
 			(project ""
 				(path "/48ddfdd8-68fa-4e63-aa18-bc113cdf8cfa/aa9739d0-05d8-4c74-a4fd-846c263eed0b"
-					(reference "#PWR0402")
-					(unit 1)
-				)
+					(reference "#PWR025")
+					(unit 1)
+				)
