File: windows/switch.kicad_sch (KiCad schematic)
At the start: 2 parts, among them CN801 39-30-1020, U801 GAQY221S

Commit message: window controller v2
Parts:
- added R2: 560, Resistor_SMD:R_0603_1608Metric, symbol Device:R
Connections:
- net GND is gone; now on net IN: U801.2
- net IN: no longer U801.1
- new net: R2.2, U801.1
- new net 5V: R2.1
Other:
- moved on the sheet: CN801, U801
Changed lines of the file:
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@@
 	(wire
 		(pts
-			(xy 78.74 35.56) (xy 69.85 35.56)
-		)
-		(stroke
-			(width 0)
-			(type default)
-		)
-	)
-	(wire
-		(pts
-			(xy 64.77 41.91) (xy 69.85 41.91)
-		)
-		(stroke
-			(width 0)
-			(type default)
-		)
-	)
-	(wire
-		(pts
-			(xy 31.75 41.91) (xy 39.37 41.91)
-		)
-		(stroke
-			(width 0)
-			(type default)
-		)
-	)
-	(wire
-		(pts
-			(xy 69.85 31.75) (xy 64.77 31.75)
-		)
-		(stroke
-			(width 0)
-			(type default)
-		)
-	)
-	(wire
-		(pts
-			(xy 31.75 31.75) (xy 39.37 31.75)
-		)
-		(stroke
-			(width 0)
-			(type default)
-		)
-	)
-	(wire
-		(pts
-			(xy 69.85 38.1) (xy 69.85 41.91)
-		)
-		(stroke
-			(width 0)
-			(type default)
-		)
-	)
-	(wire
-		(pts
-			(xy 69.85 35.56) (xy 69.85 31.75)
-		)
-		(stroke
-			(width 0)
-			(type default)
-		)
-	)
-	(wire
-		(pts
-			(xy 78.74 38.1) (xy 69.85 38.1)
+			(xy 96.52 39.37) (xy 87.63 39.37)
+		)
+		(stroke
+			(width 0)
+			(type default)
+		)
+	)
+	(wire
+		(pts
+			(xy 82.55 45.72) (xy 87.63 45.72)
+		)
+		(stroke
+			(width 0)
+			(type default)
+		)
+	)
+	(wire
+		(pts
+			(xy 50.8 35.56) (xy 57.15 35.56)
+		)
+		(stroke
+			(width 0)
+			(type default)
+		)
+	)
+	(wire
+		(pts
+			(xy 87.63 35.56) (xy 82.55 35.56)
+		)
+		(stroke
+			(width 0)
+			(type default)
+		)
+	)
+	(wire
+		(pts
+			(xy 87.63 41.91) (xy 87.63 45.72)
+		)
+		(stroke
+			(width 0)
+			(type default)
+		)
+	)
+	(wire
+		(pts
+			(xy 87.63 39.37) (xy 87.63 35.56)
+		)
+		(stroke
+			(width 0)
+			(type default)
+		)
+	)
+	(wire
+		(pts
+			(xy 38.1 35.56) (xy 43.18 35.56)
+		)
+		(stroke
+			(width 0)
+			(type default)
+		)
+	)
+	(wire
+		(pts
+			(xy 38.1 45.72) (xy 57.15 45.72)
+		)
+		(stroke
+			(width 0)
+			(type default)
+		)
+	)
+	(wire
+		(pts
+			(xy 96.52 41.91) (xy 87.63 41.91)
 		)
 		(stroke
@@
 	(hierarchical_label "IN"
 		(shape input)
-		(at 31.75 31.75 180)
+		(at 38.1 45.72 180)
 		(effects
 			(font
@@
 		)
 	)
+	(hierarchical_label "5V"
+		(shape input)
+		(at 38.1 35.56 180)
+		(effects
+			(font
+				(size 1.27 1.27)
+			)
+			(justify right)
+		)
+	)
 	(symbol
-		(lib_id "power:GND")
-		(at 31.75 41.91 0)
+		(lib_id "Device:R")
+		(at 46.99 35.56 90)
 		(unit 1)
 		(exclude_from_sim no)
@@
 		(dnp no)
 		(fields_autoplaced yes)
-		(property "Reference" "#PWR0801"
-			(at 31.75 48.26 0)
-			(effects
-				(font
-					(size 1.27 1.27)
-				)
-				(hide yes)
-			)
-		)
-		(property "Value" "GND"
-			(at 31.75 46.99 0)
-			(effects
-				(font
-					(size 1.27 1.27)
-				)
-			)
-		)
-		(property "Footprint" ""
-			(at 31.75 41.91 0)
-			(effects
-				(font
-					(size 1.27 1.27)
-				)
-				(hide yes)
-			)
-		)
-		(property "Datasheet" ""
-			(at 31.75 41.91 0)
-			(effects
-				(font
-					(size 1.27 1.27)
-				)
-				(hide yes)
-			)
-		)
-		(property "Description" "Power symbol creates a global label with name \"GND\" , ground"
-			(at 31.75 41.91 0)
+		(property "Reference" "R2"
+			(at 46.99 29.21 90)
+			(effects
+				(font
+					(size 1.27 1.27)
+				)
+			)
+		)
+		(property "Value" "560"
+			(at 46.99 31.75 90)
+			(effects
+				(font
+					(size 1.27 1.27)
+				)
+			)
+		)
+		(property "Footprint" "Resistor_SMD:R_0603_1608Metric"
+			(at 46.99 37.338 90)
+			(effects
+				(font
+					(size 1.27 1.27)
+				)
+				(hide yes)
+			)
+		)
+		(property "Datasheet" "~"
+			(at 46.99 35.56 0)
+			(effects
+				(font
+					(size 1.27 1.27)
+				)
+				(hide yes)
+			)
+		)
+		(property "Description" "Resistor"
+			(at 46.99 35.56 0)
 			(effects
 				(font
@@
 		(pin "1"
 		)
+		(pin "2"
+		)
 		(instances
-			(project "windows"
+			(project ""
 				(path "/48ddfdd8-68fa-4e63-aa18-bc113cdf8cfa/3fbbc9fa-971e-4e55-bae4-4ebcd9323906"
-					(reference "#PWR0801")
+					(reference "R2")
 					(unit 1)
 				)
 				(path "/48ddfdd8-68fa-4e63-aa18-bc113cdf8cfa/a91e3a1d-f219-4009-b0e9-cbbe40cd95e5"
-					(reference "#PWR0901")
+					(reference "R3")
 					(unit 1)
 				)
 				(path "/48ddfdd8-68fa-4e63-aa18-bc113cdf8cfa/bc2c72fb-830b-4a09-9f5e-aaaaf606b37e"
-					(reference "#PWR01001")
+					(reference "R4")
 					(unit 1)
 				)
 				(path "/48ddfdd8-68fa-4e63-aa18-bc113cdf8cfa/c6eed8fb-eaaf-47a7-809d-bebf0e2693b0"
-					(reference "#PWR01101")
+					(reference "R5")
 					(unit 1)
 				)
@@
 	(symbol
 		(lib_id "easyeda2kicad:39-30-1020")
-		(at 82.55 36.83 180)
+		(at 100.33 40.64 180)
 		(unit 1)
 		(exclude_from_sim no)
@@
 		(fields_autoplaced yes)
 		(property "Reference" "CN801"
-			(at 87.63 35.5599 0)
+			(at 105.41 39.3699 0)
 			(effects
 				(font
@@
 		)
 		(property "Value" "39-30-1020"
-			(at 87.63 38.0999 0)
+			(at 105.41 41.9099 0)
 			(effects
 				(font
@@
 		)
 		(property "Footprint" "easyeda2kicad:CONN-TH_2P-P5.50_39-30-1020"
-			(at 82.55 27.94 0)
+			(at 100.33 31.75 0)
 			(effects
 				(font
@@
 		)
 		(property "Datasheet" "https://lcsc.com/product-detail/Others_MOLEX_39-30-1020_MOLEX-39-30-1020_C240832.html"
-			(at 82.55 25.4 0)
+			(at 100.33 29.21 0)
 			(effects
 				(font
@@
 		)
 		(property "Description" ""
-			(at 82.55 36.83 0)
+			(at 100.33 40.64 0)
 			(effects
 				(font
@@
 		)
 		(property "LCSC Part" "C240832"
-			(at 82.55 22.86 0)
+			(at 100.33 26.67 0)
 			(effects
 				(font
@@
 	(symbol
 		(lib_id "easyeda2kicad:GAQY221S")
-		(at 52.07 36.83 0)
+		(at 69.85 40.64 0)
 		(unit 1)
 		(exclude_from_sim no)
@@
 		(fields_autoplaced yes)
 		(property "Reference" "U801"
-			(at 52.455 24.13 0)
+			(at 70.235 27.94 0)
 			(effects
 				(font
@@
 		)
 		(property "Value" "GAQY221S"
-			(at 52.455 26.67 0)
+			(at 70.235 30.48 0)
 			(effects
 				(font
@@
 		)
 		(property "Footprint" "easyeda2kicad:SOP-4_L4.3-W4.4-P2.54-LS7.0-BL"
-			(at 52.07 49.53 0)
+			(at 69.85 53.34 0)
 			(effects
 				(font
@@
 		)
 		(property "Datasheet" ""
-			(at 52.07 36.83 0)
+			(at 69.85 40.64 0)
 			(effects
 				(font
@@
 		)
 		(property "Description" ""
-			(at 52.07 36.83 0)
+			(at 69.85 40.64 0)
 			(effects
 				(font
@@
 		)
 		(property "LCSC Part" "C7435105"
-			(at 52.07 52.07 0)
-			(effects
-				(font
+			(at 69.85 55.88 0)
+			(effects
+				(font
