File: windows/windows.kicad_pcb (KiCad board)
At the start: 4 copper layers, 70 x 45 mm, 34 parts, among them CN1001 39-30-1020, CN1101 39-30-1020, CN201 BM04B-SRSS-TB(LF)(SN), CN301 BM04B-SRSS-TB(LF)(SN), CN401 39-30-1020, CN501 39-30-1020, CN601 39-30-1020, CN701 39-30-1020, CN801 39-30-1020, CN901 39-30-1020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

Commit message: more tweaking
Routing:
- net /i2c/VIN: track 32.6 -> 34.0 mm

Commit message: window controller v2
Parts:
- removed U102: DTS04GE, easyeda2kicad:SW-SMD_4P-L10.6-W6.9-P2.54-LS9.7_DTS04GE
- added J1: Conn_02x03_Odd_Even, Connector_PinHeader_2.54mm:PinHeader_2x03_P2.54mm_Vertical, F.Cu at (27.7, 18.5)
- added R1: 10k, Resistor_SMD:R_0603_1608Metric, F.Cu at (41.0, 23.5)
- added R2: 560, Resistor_SMD:R_0603_1608Metric, F.Cu at (60.5, 31.0)
- added R3: 560, Resistor_SMD:R_0603_1608Metric, F.Cu at (54.0, 31.0)
- added R4: 560, Resistor_SMD:R_0603_1608Metric, F.Cu at (67.0, 31.0)
- added R5: 560, Resistor_SMD:R_0603_1608Metric, F.Cu at (73.5, 31.0)
- added R6: 10k, Resistor_SMD:R_0603_1608Metric, F.Cu at (36.5, 17.5)
- added R7: 10k, Resistor_SMD:R_0603_1608Metric, F.Cu at (36.5, 19.0)
- added R8: 10k, Resistor_SMD:R_0603_1608Metric, F.Cu at (36.5, 20.5)
- added TP1: LabeledTestPoint, easyeda2kicad:LabeledTestPoint, F.Cu at (34.0, 24.0)
- added TP10: LabeledTestPoint, easyeda2kicad:LabeledTestPoint, F.Cu at (60.5, 28.5)
- added TP11: LabeledTestPoint, easyeda2kicad:LabeledTestPoint, F.Cu at (73.5, 27.0)
- added TP12: LabeledTestPoint, easyeda2kicad:LabeledTestPoint, F.Cu at (78.5, 27.0)
- added TP2: LabeledTestPoint, easyeda2kicad:LabeledTestPoint, F.Cu at (37.0, 24.0)
- added TP3: LabeledTestPoint, easyeda2kicad:LabeledTestPoint, F.Cu at (39.5, 28.5)
- added TP4: LabeledTestPoint, easyeda2kicad:LabeledTestPoint, F.Cu at (42.5, 28.5)
- added TP5: LabeledTestPoint, easyeda2kicad:LabeledTestPoint, F.Cu at (45.5, 28.5)
- added TP6: LabeledTestPoint, easyeda2kicad:LabeledTestPoint, F.Cu at (48.5, 28.5)
- added TP7: LabeledTestPoint, easyeda2kicad:LabeledTestPoint, F.Cu at (51.5, 28.5)
- added TP8: LabeledTestPoint, easyeda2kicad:LabeledTestPoint, F.Cu at (54.5, 28.5)
- added TP9: LabeledTestPoint, easyeda2kicad:LabeledTestPoint, F.Cu at (57.5, 28.5)
- moved U1001 3.40 mm to (67.0, 36.5)
- moved U1101 3.40 mm to (73.5, 36.5)
- moved U801 3.40 mm to (60.6, 36.5)
- moved U901 3.40 mm to (54.0, 36.5)
Connections:
- U1001 pad 1: /switch2/IN -> Net-(R4-Pad2)
- U1001 pad 2: GND -> /switch2/IN
- U101 pad 4: unconnected-(U101-~{RESET}-Pad4) -> Net-(U101-~{RESET})
- U101 pad 7: unconnected-(U101-INT-Pad7) -> Net-(U101-INT)
- U1101 pad 1: /switch3/IN -> Net-(R5-Pad2)
- U1101 pad 2: GND -> /switch3/IN
- U801 pad 1: /switch1/IN -> Net-(R2-Pad2)
- U801 pad 2: GND -> /switch1/IN
- U901 pad 1: /switch/IN -> Net-(R3-Pad2)
- U901 pad 2: GND -> /switch/IN
Routing:
- net Net-(U101-INT): track 0.00 -> 17.3 mm
- net Net-(U101-~{RESET}): track 0.00 -> 15.5 mm
- net Net-(J1-Pin_6): track 15.1 -> 22.3 mm
- net /i2c/VIN: track 34.0 -> 38.3 mm, vias 11 -> 15
- net GND: track 16.2 -> 19.7 mm, vias 22 -> 20
- net Net-(CN1101-Pad2): track 8.63 -> 5.23 mm
- net Net-(CN901-Pad2): track 8.56 -> 5.16 mm
- net Net-(CN801-Pad2): track 8.54 -> 5.14 mm
- net Net-(CN1001-Pad2): track 8.61 -> 5.21 mm
- net Net-(CN1001-Pad1): track 14.7 -> 11.8 mm
- net Net-(CN801-Pad1): track 14.6 -> 11.8 mm
- net /switch/IN: track 8.12 -> 10.9 mm
- net Net-(CN901-Pad1): track 14.6 -> 11.8 mm
- net Net-(J1-Pin_4): track 19.4 -> 22.0 mm
- net Net-(CN1101-Pad1): track 14.7 -> 12.2 mm
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Other:
- board text added: "5"
- board text added: "6"
- board text added: "7"
- board text added: "8"
- board text added: "Window Controller V0.2"
- board text removed: "Window Controller V0.1"
