File: roomsensor/i2c.kicad_sch (KiCad schematic)
At the start: 5 parts, among them CN601 BM04B-SRSS-TB(LF)(SN), Q601 BSS138, Q602 BSS138

Commit message: roomsenor v2.2
Parts:
- renumbered CN601 to CN1, Q602 to Q1, Q601 to Q2, R601 to R7, R602 to R8
Changed lines of the file:
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@@
 (kicad_sch
-	(version 20231120)
+	(version 20250114)
 	(generator "eeschema")
-	(generator_version "8.0")
+	(generator_version "9.0")
 	(paper "A4")
 	(junction
@@
 	(label "I2C.SCL"
 		(at 36.83 45.72 0)
-		(fields_autoplaced yes)
 		(effects
 			(font
@@
 	(label "I2C.SDA"
 		(at 38.1 36.83 0)
-		(fields_autoplaced yes)
 		(effects
 			(font
@@
 		(shape input)
 		(at 30.48 33.02 180)
-		(fields_autoplaced yes)
 		(effects
 			(font
@@
 		(shape input)
 		(at 48.26 25.4 180)
-		(fields_autoplaced yes)
 		(effects
 			(font
@@
 		(shape input)
 		(at 48.26 19.05 180)
-		(fields_autoplaced yes)
 		(effects
 			(font
@@
 		(dnp no)
 		(fields_autoplaced yes)
-		(property "Reference" "#PWR0601"
+		(property "Reference" "#PWR011"
 			(at 109.22 31.75 0)
 			(effects
@@
 			(project "roomsensor"
 				(path "/48ddfdd8-68fa-4e63-aa18-bc113cdf8cfa/9bbd6b58-2c5b-4ba0-9255-412ba0fc4a43"
-					(reference "#PWR0601")
+					(reference "#PWR011")
 					(unit 1)
 				)
@@
 		(dnp no)
 		(fields_autoplaced yes)
-		(property "Reference" "CN601"
+		(property "Reference" "CN1"
 			(at 132.08 35.5599 0)
 			(effects
@@
 			(project "roomsensor"
 				(path "/48ddfdd8-68fa-4e63-aa18-bc113cdf8cfa/9bbd6b58-2c5b-4ba0-9255-412ba0fc4a43"
-					(reference "CN601")
+					(reference "CN1")
 					(unit 1)
 				)
@@
 		(dnp no)
 		(fields_autoplaced yes)
-		(property "Reference" "R602"
+		(property "Reference" "R8"
 			(at 95.25 29.2099 0)
 			(effects
@@
 			(project "roomsensor"
 				(path "/48ddfdd8-68fa-4e63-aa18-bc113cdf8cfa/9bbd6b58-2c5b-4ba0-9255-412ba0fc4a43"
-					(reference "R602")
+					(reference "R8")
 					(unit 1)
 				)
@@
 		(dnp no)
 		(fields_autoplaced yes)
-		(property "Reference" "R601"
+		(property "Reference" "R7"
 			(at 82.55 29.2099 0)
 			(effects
@@
 			(project "roomsensor"
 				(path "/48ddfdd8-68fa-4e63-aa18-bc113cdf8cfa/9bbd6b58-2c5b-4ba0-9255-412ba0fc4a43"
-					(reference "R601")
+					(reference "R7")
 					(unit 1)
 				)
@@
 		(dnp no)
 		(fields_autoplaced yes)
-		(property "Reference" "Q601"
+		(property "Reference" "Q2"
 			(at 69.85 40.64 90)
 			(effects
@@
 			(project "roomsensor"
 				(path "/48ddfdd8-68fa-4e63-aa18-bc113cdf8cfa/9bbd6b58-2c5b-4ba0-9255-412ba0fc4a43"
-					(reference "Q601")
+					(reference "Q2")
 					(unit 1)
 				)
@@
 		(dnp no)
 		(fields_autoplaced yes)
-		(property "Reference" "Q602"
+		(property "Reference" "Q1"
 			(at 59.69 49.53 90)
 			(effects
@@
 			(project "roomsensor"
 				(path "/48ddfdd8-68fa-4e63-aa18-bc113cdf8cfa/9bbd6b58-2c5b-4ba0-9255-412ba0fc4a43"
-					(reference "Q602")
+					(reference "Q1")
 					(unit 1)
 				)
