File: roomsensor/mic.kicad_sch (KiCad schematic)
At the start: 3 parts, among them U301 BME280

Commit message: more work on roomsensor
Parts:
- removed C301, C302: 100nF, Capacitor_SMD:C_0603_1608Metric, symbol Device:C
- removed U301: BME280, Package_LGA:Bosch_LGA-8_2.5x2.5mm_P0.65mm_ClockwisePinNumbering, symbol Sensor:BME280
- added C1001: 100nF, Capacitor_SMD:C_0603_1608Metric, symbol Device:C
- added U1001: ICS-43434_C5656610, easyeda2kicad:MIC-SMD_6P-L3.5-W2.7-P0.90-BL, symbol easyeda2kicad:ICS-43434_C5656610
Connections:
- net 3v3: now also C1001.1, U1001.5 (VDD)
- net GND: now also C1001.2, U1001.2 (LR), U1001.3 (GND)
- new net I2S.SCK: U1001.4 (SCK)
- new net I2S.SD: U1001.6 (SD)
- new net I2S.WS: U1001.1 (WS)

Commit message: roomsenor v2.2
Parts:
- renumbered C1001 to C21, U1001 to U7
Changed lines of the file:
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@@
 (kicad_sch
-	(version 20231120)
+	(version 20250114)
 	(generator "eeschema")
-	(generator_version "8.0")
+	(generator_version "9.0")
 	(paper "A4")
 	(junction
@@
 	(label "I2S.WS"
 		(at 60.96 46.99 0)
-		(fields_autoplaced yes)
 		(effects
 			(font
@@
 	(label "I2S.SD"
 		(at 60.96 50.8 0)
-		(fields_autoplaced yes)
 		(effects
 			(font
@@
 	(label "I2S.SCK"
 		(at 60.96 43.18 0)
-		(fields_autoplaced yes)
 		(effects
 			(font
@@
 		(shape input)
 		(at 73.66 40.64 0)
-		(fields_autoplaced yes)
 		(effects
 			(font
@@
 		(shape input)
 		(at 25.4 33.02 180)
-		(fields_autoplaced yes)
 		(effects
 			(font
@@
 		(dnp no)
 		(fields_autoplaced yes)
-		(property "Reference" "C1001"
+		(property "Reference" "C21"
 			(at 34.29 35.5599 0)
 			(effects
@@
 			(project ""
 				(path "/48ddfdd8-68fa-4e63-aa18-bc113cdf8cfa/c4514872-6898-4930-85b8-95c1964554a5"
-					(reference "C1001")
+					(reference "C21")
 					(unit 1)
 				)
@@
 		(on_board yes)
 		(dnp no)
-		(property "Reference" "U1001"
+		(property "Reference" "U7"
 			(at 51.054 25.654 0)
 			(effects
@@
 			(project ""
 				(path "/48ddfdd8-68fa-4e63-aa18-bc113cdf8cfa/c4514872-6898-4930-85b8-95c1964554a5"
-					(reference "U1001")
+					(reference "U7")
 					(unit 1)
 				)
@@
 		(dnp no)
 		(fields_autoplaced yes)
-		(property "Reference" "#PWR01001"
+		(property "Reference" "#PWR014"
 			(at 50.8 68.58 0)
 			(effects
@@
 			(project ""
 				(path "/48ddfdd8-68fa-4e63-aa18-bc113cdf8cfa/c4514872-6898-4930-85b8-95c1964554a5"
-					(reference "#PWR01001")
+					(reference "#PWR014")
 					(unit 1)
 				)
