File: roomsensor/pir_d.kicad_sch (KiCad schematic)
At the start: 2 parts, among them U1301 SM03B-SRSS-TB(LF)(SN)(P)

Commit message: sensor v2.1
Parts:
- removed R1301: 4.7k, Resistor_SMD:R_0603_1608Metric, symbol Device:R
- removed U1301: SM03B-SRSS-TB(LF)(SN)(P), easyeda2kicad:CONN-SMD_SM03B-SRSS-TB-LF-SN-P, symbol easyeda2kicad:SM03B-SRSS-TB(LF)(SN)(P)
- added R2001: 10k, Resistor_SMD:R_0603_1608Metric, symbol Device:R
- added TP1901: LabeledTestPoint, easyeda2kicad:LabeledTestPoint, symbol easyeda2kicad:LabeledTestPoint
- added U2001: EKMC1601112, easyeda2kicad:SENSOR-TH_EKMC1601111, symbol easyeda2kicad:EKMC1601112
Connections:
- net 3v3: now also R2001.1, U2001.1 (VDD)
- net GND: now also U2001.3 (GND)
- new net VOUT: R2001.2, TP1901.1, U2001.2 (OUT)

Commit message: roomsenor v2.2
Parts:
- added C24: 1uF, Capacitor_SMD:C_0603_1608Metric, symbol Device:C
- added C25: 100nF, Capacitor_SMD:C_0603_1608Metric, symbol Device:C
- R15: renamed from R2001; value 10k -> 100k
- renumbered TP1901 to TP4, U2001 to U10
Connections:
- net 3v3: now also C24.1, C25.1; no longer R15.1
- net GND: now also R15.2, C24.2, C25.2
- net VOUT: now also R15.1; no longer R15.2
Other:
- moved on the sheet: R15, U10
