File: roomsensor/lux.kicad_sch (KiCad schematic)
At the start: 3 parts, among them U2002 OPT3001DNPR

Commit message: roomsenor v2.2
Parts:
- renumbered C2001 to C26, TP2001 to TP5, U2002 to U11
Changed lines of the file:
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@@
 (kicad_sch
-	(version 20231120)
+	(version 20250114)
 	(generator "eeschema")
-	(generator_version "8.0")
+	(generator_version "9.0")
 	(paper "A4")
 	(junction
@@
 		(shape input)
 		(at 97.79 34.29 0)
-		(fields_autoplaced yes)
 		(effects
 			(font
@@
 		(shape input)
 		(at 25.4 36.83 180)
-		(fields_autoplaced yes)
 		(effects
 			(font
@@
 		(dnp no)
 		(fields_autoplaced yes)
-		(property "Reference" "#PWR02002"
+		(property "Reference" "#PWR055"
 			(at 45.72 58.42 0)
 			(effects
@@
 			(project ""
 				(path "/48ddfdd8-68fa-4e63-aa18-bc113cdf8cfa/2937f9cc-cdae-43bf-bd0c-68c845d5f8b1"
-					(reference "#PWR02002")
+					(reference "#PWR055")
 					(unit 1)
 				)
@@
 		(dnp no)
 		(fields_autoplaced yes)
-		(property "Reference" "TP2001"
+		(property "Reference" "TP5"
 			(at 89.408 39.37 0)
 			(effects
@@
 			(project ""
 				(path "/48ddfdd8-68fa-4e63-aa18-bc113cdf8cfa/2937f9cc-cdae-43bf-bd0c-68c845d5f8b1"
-					(reference "TP2001")
+					(reference "TP5")
 					(unit 1)
 				)
@@
 		(dnp no)
 		(fields_autoplaced yes)
-		(property "Reference" "U2002"
+		(property "Reference" "U11"
 			(at 62.23 29.21 0)
 			(effects
@@
 			(project ""
 				(path "/48ddfdd8-68fa-4e63-aa18-bc113cdf8cfa/2937f9cc-cdae-43bf-bd0c-68c845d5f8b1"
-					(reference "U2002")
+					(reference "U11")
 					(unit 1)
 				)
@@
 		(dnp no)
 		(fields_autoplaced yes)
-		(property "Reference" "C2001"
+		(property "Reference" "C26"
 			(at 35.56 39.3699 0)
 			(effects
@@
 			(project ""
 				(path "/48ddfdd8-68fa-4e63-aa18-bc113cdf8cfa/2937f9cc-cdae-43bf-bd0c-68c845d5f8b1"
-					(reference "C2001")
+					(reference "C26")
 					(unit 1)
 				)
