File: roomsensor/roomsensor.kicad_sch (KiCad schematic)
At the start: 0 parts

Commit message: more work on roomsensor
Parts:
- added C101, C102: 22uF, Capacitor_SMD:C_Elec_5x5.8, symbol Device:C_Polarized
- added H101, H102, H103, H104: MountingHole_Pad, MountingHole:MountingHole_3.2mm_M3_Pad_Via, symbol Mechanical:MountingHole_Pad
Connections:
- net +5V: now also C101.1, C102.1
- new net GND: C101.2, C102.2, H101.1, H102.1, H103.1, H104.1
Other:
- added sheet mic (mic.kicad_sch)
- added sheet pira (pira.kicad_sch)
- sheet esp32 ports: added I2C{SDA,SCL}, USB{DP,DN}; removed I2C{SDA, SCL}

Commit message: roomsensor v2.0
Other:
- added sheet accel (accel.kicad_sch)
- added sheet i2c-horiz (i2ch.kicad_sch)
- added sheet temp (temp.kicad_sch)
- sheet bme680 ports: added 3v3; removed none
- sheet esp32 ports: added I2S{SCK,WS,SD}, accel, temp; removed none
- sheet mic ports: added 3v3, I2S{SCK,WS,SD}; removed none
- moved on the sheet: C101, C102, H101, H102, H103, H104

Commit message: sensor v2.1
Parts:
- added TP101, TP102: LabeledTestPoint, easyeda2kicad:LabeledTestPoint, symbol easyeda2kicad:LabeledTestPoint
Connections:
- net +5V: now also TP101.1
- net 3v3/VOUT: now also TP102.1
- no-connect marks 0 -> 1
Other:
- removed sheet pira
- added sheet lux (lux.kicad_sch)
- added sheet pir_d (pir_d.kicad_sch)

Commit message: roomsenor v2.2
Parts:
- removed C101, C102: 22uF, Capacitor_SMD:C_Elec_5x5.8, symbol Device:C_Polarized
- added C2: 47uF, Capacitor_SMD:CP_Elec_6.3x5.9, symbol Device:C_Polarized
- renumbered H101 to H1, H102 to H2, H103 to H3, H104 to H4, TP101 to TP1, TP102 to TP2
Connections:
- net +5V: now also C2.1
- net GND: now also C2.2

Commit message: WIP roomsensor 2.3
Parts:
- added H5, H6: MountingHole_Pad, MountingHole:MountingHole_3.2mm_M3_Pad_Via, symbol Mechanical:MountingHole_Pad
- added RF1, RF2: 73412-0110, easyeda2kicad:ANT-SMD_73412-0110, symbol easyeda2kicad:73412-0110
Connections:
- net +5V: now also RF2.2 (SIG)
- net 3v3/VOUT: now also RF1.2 (SIG)
- net GND: now also H5.1, H6.1, RF1.1 (GND), RF1.3 (GND), RF1.4 (GND), RF2.1 (GND), RF2.3 (GND), RF2.4 (GND)
Other:
- removed sheet i2c
- added sheet i2c-horiz1 (i2ch.kicad_sch)
- moved on the sheet: C2, H1, H2, H3, H4

Commit message: roomsensor v2.3
Other:
- sheet esp32 ports: added 5V; removed none
Changed lines of the file:
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@@
+	)
+	(junction
+		(at 52.07 46.99)
+		(diameter 0)
+		(color 0 0 0 0)
 	)
 	(junction
@@
 	(wire
 		(pts
+			(xy 52.07 46.99) (xy 52.07 54.61)
+		)
+		(stroke
+			(width 0)
+			(type default)
+		)
+	)
+	(wire
+		(pts
 			(xy 86.36 44.45) (xy 101.6 44.45)
 		)
@@
 	(wire
 		(pts
+			(xy 91.44 46.99) (xy 52.07 46.99)
+		)
+		(stroke
+			(width 0)
+			(type default)
+		)
+	)
+	(wire
+		(pts
 			(xy 53.34 106.68) (xy 60.96 106.68)
 		)
@@
 	(wire
 		(pts
-			(xy 52.07 44.45) (xy 52.07 54.61)
+			(xy 52.07 44.45) (xy 52.07 46.99)
 		)
 		(stroke
@@
 	(wire
 		(pts
+			(xy 106.68 53.34) (xy 91.44 53.34)
+		)
+		(stroke
+			(width 0)
+			(type default)
+		)
+	)
+	(wire
+		(pts
 			(xy 109.22 101.6) (xy 99.06 101.6)
 		)
@@
 		(pts
 			(xy 78.74 73.66) (xy 78.74 80.01)
+		)
+		(stroke
+			(width 0)
+			(type default)
+		)
+	)
+	(wire
+		(pts
+			(xy 91.44 53.34) (xy 91.44 46.99)
 		)
 		(stroke
@@
 			)
 		)
+		(pin "5V" input
+			(at 106.68 53.34 180)
+			(effects
+				(font
+					(size 1.27 1.27)
+				)
+				(justify left)
+			)
+		)
