File: locks/locks.kicad_sch (KiCad schematic)
At the start: 36 parts, among them CN1 39-30-1020, J1 Conn_02x03_Odd_Even, J2 Conn_02x04_Odd_Even, U1 MCP23008-xML, U2 ADS1115IDGS

Commit message: last tweaks to locks
Parts:
- J2: LCSC Part C5383105 -> (none)
Changed lines of the file:
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@@
 	(wire
 		(pts
-			(xy 182.88 113.03) (xy 228.6 113.03)
+			(xy 195.58 113.03) (xy 228.6 113.03)
 		)
 		(stroke
@@
 			)
 		)
-		(property "LCSC Part" "C5383105"
-			(at 255.27 129.54 0)
-			(effects
-				(font
-					(size 1.27 1.27)
-				)
-				(hide yes)
-			)
-		)
 		(pin "1"
 		)
@@
 		)
 		(property "Label" "SDA"
-			(at 58.166 80.772 0)
+			(at 59.69 80.7719 0)
 			(effects
 				(font
@@
 		)
 		(property "Label" "SCL"
-			(at 58.166 66.548 0)
+			(at 59.69 66.5479 0)
 			(effects
 				(font
@@
 		)
 		(pin "IS" input
-			(at 182.88 113.03 180)
+			(at 195.58 113.03 0)
 			(effects
 				(font
 					(size 1.27 1.27)
 				)
-				(justify left)
+				(justify right)
 			)
 		)
