File: air/air.kicad_sch (KiCad schematic)
At the start: 8 parts, among them CN1 SM06B-GHS-TB(LF)(SN), U1 3SP-H2S-50_110-304, U2 SCD41-D-R2, U3 ADS1115IDGS

Commit message: first version of air sensor
Parts:
- removed CN1: SM06B-GHS-TB(LF)(SN), easyeda2kicad:CONN-TH_SM06B-GHS-TB-LF-SN, symbol easyeda2kicad:SM06B-GHS-TB(LF)(SN)
- removed U1: 3SP-H2S-50_110-304, Sensor:SPEC_110-xxx_SMD-10Pin_20x20mm_P4.0mm, symbol Sensor_Gas:3SP-H2S-50_110-304
- removed U2: SCD41-D-R2, Sensor:Sensirion_SCD4x-1EP_10.1x10.1mm_P1.25mm_EP4.8x4.8mm, symbol Sensor_Gas:SCD41-D-R2
- removed U3: ADS1115IDGS, Package_SO:TSSOP-10_3x3mm_P0.5mm, symbol Analog_ADC:ADS1115IDGS
Other:
- added sheet 3v3 (3v3.kicad_sch)
- added sheet scd41 (scd41.kicad_sch)
- added sheet sen55 (sen55.kicad_sch)
- added sheet spec_gas (spec_gas.kicad_sch)
- sheet i2c-horiz ports: added 5V; removed VCC

Commit message: air add on v0.1
Other:
- sheet i2c-horiz ports: added 3v3; removed 3V3
Changed lines of the file:
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@@
 			)
 		)
-		(pin "3V3" input
-			(at 39.37 68.58 0)
+		(pin "5V" input
+			(at 39.37 59.69 0)
 			(effects
 				(font
@@
 			)
 		)
-		(pin "5V" input
-			(at 39.37 59.69 0)
+		(pin "3v3" input
+			(at 39.37 68.58 0)
 			(effects
 				(font

Commit message: air v0.2
Parts:
- added RF101, RF102: 73412-0110, easyeda2kicad:ANT-SMD_73412-0110, symbol easyeda2kicad:73412-0110
- renumbered H1 to H101, H2 to H102, H3 to H103, H4 to H104
Connections:
- net 3v3/VIN: now also RF102.2 (SIG)
- net GND: now also RF101.1 (GND), RF101.3 (GND), RF101.4 (GND), RF102.1 (GND), RF102.3 (GND), RF102.4 (GND)
- new net 3v4/VOUT: RF101.2 (SIG)
Other:
- added sheet 3v4 (3v3.kicad_sch)
