File: air/i2ch.kicad_sch (KiCad schematic)
At the start: 5 parts, among them CN2 SM04B-SRSS-TB (LF)(SN), Q3 BSS138, Q4 BSS138

Commit message: first version of air sensor
Parts:
- added R4, R5: 4.7k, Resistor_SMD:R_0603_1608Metric, symbol Device:R
- added TP10, TP11, TP8, TP9: LabeledTestPoint, easyeda2kicad:LabeledTestPoint, symbol easyeda2kicad:LabeledTestPoint
- R6: renamed from R11; now not fitted; now left out of the parts list
- R7: renamed from R12; now not fitted; now left out of the parts list
- renumbered Q3 to Q1, Q4 to Q2
Connections:
- net 3V3: now also R4.1, R5.1
- net I2C.SCL: now also R4.2, TP8.1
- net I2C.SDA: now also R5.2, TP9.1
- net at CN2.4, Q2.3 (D), R6.2: now also TP10.1
- net at CN2.3, Q1.3 (D), R7.2: now also TP11.1
- net VCC renamed 5V

Commit message: air add on v0.1
Connections:
- net 3V3 renamed 3v3
Changed lines of the file:
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@@
 		)
 	)
-	(hierarchical_label "3V3"
+	(hierarchical_label "3v3"
 		(shape input)
 		(at 53.34 53.34 180)

Commit message: air v0.2
Parts:
- added C701: 10uF, Capacitor_SMD:C_0603_1608Metric, symbol Device:C
- added C702: 100nF, Capacitor_SMD:C_0603_1608Metric, symbol Device:C
- TP701: renamed from TP8; Label SCL3v3 -> SCL
- TP703: renamed from TP9; Label SDA3v3 -> SDA
- renumbered CN2 to CN701, Q2 to Q701, Q1 to Q702, R4 to R701, R5 to R702, R6 to R703, R7 to R704, TP10 to TP702, TP11 to TP704
Connections:
- net 5V: now also C701.1, C702.1; no longer CN701.5, CN701.6
- net GND: now also CN701.5, CN701.6, C701.2, C702.2
- net scl5v: now reaches CN701.4, Q701.3 (D), R703.2, TP702.1
- net sda5v: now reaches CN701.3, Q702.3 (D), R704.2, TP704.1
