File: air/scd41.kicad_sch (KiCad schematic)
At the start: 4 parts, among them U1 SCD41-D-R2

Commit message: air v0.2
Parts:
- added C501, C502: 10uF, Capacitor_SMD:C_0603_1608Metric, symbol Device:C
- renumbered C12 to C503, C13 to C504, C11 to C505, U1 to U501
Connections:
- net GND: now also C501.2, C502.2
- net VCC: now also C501.1, C502.1
Other:
- moved on the sheet: C503, C504, C505, U501
