File: air/sen55.kicad_sch (KiCad schematic)
At the start: 3 parts, among them CN1 SM06B-GHS-TB(LF)(SN)

Commit message: air add on v0.1
Connections:
- no-connect marks 0 -> 3
Changed lines of the file:
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@@
 		(color 0 0 0 0)
+	)
+	(no_connect
+		(at 88.9 67.31)
+	)
+	(no_connect
+		(at 104.14 54.61)
+	)
+	(no_connect
+		(at 104.14 67.31)
 	)
 	(bus_entry

Commit message: air v0.2
Parts:
- added C601, C602: 10uF, Capacitor_SMD:C_0603_1608Metric, symbol Device:C
- renumbered C15 to C603, C14 to C604, CN1 to CN601
Connections:
- net 5V: now also C601.1, C602.1
- net GND: now also C601.2, C602.2
Changed lines of the file:
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@@
 	(paper "A4")
 	(junction
+		(at 45.72 46.99)
+		(diameter 0)
+		(color 0 0 0 0)
+	)
+	(junction
+		(at 45.72 39.37)
+		(diameter 0)
+		(color 0 0 0 0)
+	)
+	(junction
 		(at 69.85 39.37)
 		(diameter 0)
@@
 	(junction
 		(at 81.28 64.77)
+		(diameter 0)
+		(color 0 0 0 0)
+	)
+	(junction
+		(at 58.42 46.99)
+		(diameter 0)
+		(color 0 0 0 0)
+	)
+	(junction
+		(at 33.02 39.37)
 		(diameter 0)
 		(color 0 0 0 0)
@@
 	(wire
 		(pts
+			(xy 33.02 39.37) (xy 45.72 39.37)
+		)
+		(stroke
+			(width 0)
+			(type default)
+		)
+	)
+	(wire
+		(pts
 			(xy 81.28 64.77) (xy 81.28 71.12)
 		)
@@
 	(wire
 		(pts
+			(xy 45.72 46.99) (xy 58.42 46.99)
+		)
+		(stroke
+			(width 0)
+			(type default)
+		)
+	)
+	(wire
+		(pts
 			(xy 88.9 57.15) (xy 81.28 57.15)
 		)
@@
 	(wire
 		(pts
+			(xy 33.02 46.99) (xy 45.72 46.99)
+		)
+		(stroke
+			(width 0)
+			(type default)
+		)
+	)
+	(wire
+		(pts
 			(xy 88.9 64.77) (xy 81.28 64.77)
 		)
@@
 	(wire
 		(pts
-			(xy 46.99 39.37) (xy 58.42 39.37)
+			(xy 25.4 39.37) (xy 33.02 39.37)
 		)
 		(stroke
@@
 		(pts
 			(xy 69.85 39.37) (xy 80.01 39.37)
+		)
+		(stroke
+			(width 0)
+			(type default)
+		)
+	)
+	(wire
+		(pts
+			(xy 45.72 39.37) (xy 58.42 39.37)
 		)
 		(stroke
@@
 	(hierarchical_label "5V"
 		(shape input)
-		(at 46.99 39.37 180)
+		(at 25.4 39.37 180)
 		(effects
 			(font
@@
 		(dnp no)
 		(fields_autoplaced yes)
-		(property "Reference" "C14"
+		(property "Reference" "C604"
 			(at 73.66 41.9099 0)
 			(effects
@@
 			(project ""
 				(path "/48ddfdd8-68fa-4e63-aa18-bc113cdf8cfa/db93cb5e-81fc-4bc4-888d-4d44a7d318b5"
-					(reference "C14")
+					(reference "C604")
 					(unit 1)
 				)
@@
 		(dnp no)
 		(fields_autoplaced yes)
-		(property "Reference" "#PWR09"
+		(property "Reference" "#PWR0601"
 			(at 81.28 77.47 0)
 			(effects
@@
 			(project ""
 				(path "/48ddfdd8-68fa-4e63-aa18-bc113cdf8cfa/db93cb5e-81fc-4bc4-888d-4d44a7d318b5"
-					(reference "#PWR09")
+					(reference "#PWR0601")
 					(unit 1)
 				)
@@
 		(dnp no)
 		(fields_autoplaced yes)
-		(property "Reference" "CN1"
+		(property "Reference" "CN601"
 			(at 96.52 46.99 0)
 			(effects
@@
 			(project "air"
 				(path "/48ddfdd8-68fa-4e63-aa18-bc113cdf8cfa/db93cb5e-81fc-4bc4-888d-4d44a7d318b5"
-					(reference "CN1")
+					(reference "CN601")
+					(unit 1)
+				)
+			)
+		)
+	)
+	(symbol
+		(lib_id "Device:C")
+		(at 33.02 43.18 0)
+		(unit 1)
+		(exclude_from_sim no)
+		(in_bom yes)
+		(on_board yes)
+		(dnp no)
+		(fields_autoplaced yes)
+		(property "Reference" "C601"
+			(at 36.83 41.9099 0)
+			(effects
+				(font
+					(size 1.27 1.27)
+				)
+				(justify left)
+			)
+		)
+		(property "Value" "10uF"
+			(at 36.83 44.4499 0)
+			(effects
+				(font
+					(size 1.27 1.27)
+				)
+				(justify left)
+			)
+		)
+		(property "Footprint" "Capacitor_SMD:C_0603_1608Metric"
+			(at 33.9852 46.99 0)
+			(effects
+				(font
+					(size 1.27 1.27)
+				)
+				(hide yes)
+			)
+		)
+		(property "Datasheet" "~"
+			(at 33.02 43.18 0)
+			(effects
+				(font
+					(size 1.27 1.27)
+				)
+				(hide yes)
+			)
+		)
+		(property "Description" "Unpolarized capacitor"
+			(at 33.02 43.18 0)
+			(effects
+				(font
+					(size 1.27 1.27)
+				)
+				(hide yes)
+			)
+		)
+		(pin "1"
+		)
+		(pin "2"
+		)
+		(instances
+			(project "air"
+				(path "/48ddfdd8-68fa-4e63-aa18-bc113cdf8cfa/db93cb5e-81fc-4bc4-888d-4d44a7d318b5"
+					(reference "C601")
+					(unit 1)
+				)
+			)
+		)
+	)
+	(symbol
+		(lib_id "Device:C")
+		(at 45.72 43.18 0)
+		(unit 1)
+		(exclude_from_sim no)
+		(in_bom yes)
+		(on_board yes)
+		(dnp no)
+		(fields_autoplaced yes)
+		(property "Reference" "C602"
+			(at 49.53 41.9099 0)
+			(effects
+				(font
+					(size 1.27 1.27)
+				)
+				(justify left)
+			)
+		)
+		(property "Value" "10uF"
+			(at 49.53 44.4499 0)
+			(effects
+				(font
+					(size 1.27 1.27)
+				)
+				(justify left)
+			)
+		)
+		(property "Footprint" "Capacitor_SMD:C_0603_1608Metric"
+			(at 46.6852 46.99 0)
+			(effects
+				(font
+					(size 1.27 1.27)
+				)
+				(hide yes)
+			)
+		)
+		(property "Datasheet" "~"
+			(at 45.72 43.18 0)
+			(effects
+				(font
+					(size 1.27 1.27)
+				)
+				(hide yes)
+			)
+		)
+		(property "Description" "Unpolarized capacitor"
+			(at 45.72 43.18 0)
+			(effects
+				(font
+					(size 1.27 1.27)
+				)
+				(hide yes)
+			)
+		)
+		(pin "1"
+		)
+		(pin "2"
+		)
+		(instances
+			(project "air"
+				(path "/48ddfdd8-68fa-4e63-aa18-bc113cdf8cfa/db93cb5e-81fc-4bc4-888d-4d44a7d318b5"
+					(reference "C602")
 					(unit 1)
 				)
@@
 		(dnp no)
 		(fields_autoplaced yes)
-		(property "Reference" "C15"
+		(property "Reference" "C603"
 			(at 62.23 41.9099 0)
 			(effects
@@
 			(project "air"
 				(path "/48ddfdd8-68fa-4e63-aa18-bc113cdf8cfa/db93cb5e-81fc-4bc4-888d-4d44a7d318b5"
-					(reference "C15")
+					(reference "C603")
 					(unit 1)
 				)
