File: leds/hi_amp/3v3.kicad_sch (KiCad schematic)
At the start: 6 parts, among them U7 TPS73733DCQ_C5220270

Commit message: WIP hi_amp leds
Parts:
- renumbered C24 to C13, C25 to C14, C26 to C15, C27 to C16, R23 to R15, U7 to U4
Changed lines of the file:
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@@
 		(dnp no)
 		(fields_autoplaced yes)
-		(property "Reference" "C25"
+		(property "Reference" "C14"
 			(at 88.9 77.4699 0)
 			(effects
@@
 			(project "espamp"
 				(path "/48ddfdd8-68fa-4e63-aa18-bc113cdf8cfa/ff982210-6c86-422a-a66b-20bff67bd030"
-					(reference "C25")
+					(reference "C14")
 					(unit 1)
 				)
@@
 		(dnp no)
 		(fields_autoplaced yes)
-		(property "Reference" "R23"
+		(property "Reference" "R15"
 			(at 90.17 55.88 90)
 			(effects
@@
 			(project "espamp"
 				(path "/48ddfdd8-68fa-4e63-aa18-bc113cdf8cfa/ff982210-6c86-422a-a66b-20bff67bd030"
-					(reference "R23")
+					(reference "R15")
 					(unit 1)
 				)
@@
 		(dnp no)
 		(fields_autoplaced yes)
-		(property "Reference" "C26"
+		(property "Reference" "C15"
 			(at 119.38 71.1199 0)
 			(effects
@@
 			(project "espamp"
 				(path "/48ddfdd8-68fa-4e63-aa18-bc113cdf8cfa/ff982210-6c86-422a-a66b-20bff67bd030"
-					(reference "C26")
+					(reference "C15")
 					(unit 1)
 				)
@@
 		(on_board yes)
 		(dnp no)
-		(property "Reference" "U7"
+		(property "Reference" "U4"
 			(at 108.712 64.262 0)
 			(effects
@@
 			(project "espamp"
 				(path "/48ddfdd8-68fa-4e63-aa18-bc113cdf8cfa/ff982210-6c86-422a-a66b-20bff67bd030"
-					(reference "U7")
+					(reference "U4")
 					(unit 1)
 				)
@@
 		(dnp no)
 		(fields_autoplaced yes)
-		(property "Reference" "#PWR029"
+		(property "Reference" "#PWR017"
 			(at 110.49 90.17 0)
 			(effects
@@
 			(project ""
 				(path "/48ddfdd8-68fa-4e63-aa18-bc113cdf8cfa/ff982210-6c86-422a-a66b-20bff67bd030"
-					(reference "#PWR029")
+					(reference "#PWR017")
 					(unit 1)
 				)
@@
 		(dnp no)
 		(fields_autoplaced yes)
-		(property "Reference" "C27"
+		(property "Reference" "C16"
 			(at 132.08 71.1199 0)
 			(effects
@@
 			(project "espamp"
 				(path "/48ddfdd8-68fa-4e63-aa18-bc113cdf8cfa/ff982210-6c86-422a-a66b-20bff67bd030"
-					(reference "C27")
+					(reference "C16")
 					(unit 1)
 				)
@@
 		(dnp no)
 		(fields_autoplaced yes)
-		(property "Reference" "C24"
+		(property "Reference" "C13"
 			(at 78.74 71.1199 0)
 			(effects
@@
 			(project "espamp"
 				(path "/48ddfdd8-68fa-4e63-aa18-bc113cdf8cfa/ff982210-6c86-422a-a66b-20bff67bd030"
-					(reference "C24")
-					(unit 1)
-				)
+					(reference "C13")
+					(unit 1)
+				)
