File: moisture/i2ch.kicad_sch (KiCad schematic)
At the start: 5 parts, among them CN2 SM04B-SRSS-TB (LF)(SN), Q3 BSS138, Q4 BSS138

Commit message: WIP
Connections:
- net 5V: no longer CN2.5, CN2.6
Changed lines of the file:
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@@
-	)
-	(junction
-		(at 148.59 76.2)
-		(diameter 0)
-		(color 0 0 0 0)
-	)
-	(junction
-		(at 148.59 66.04)
-		(diameter 0)
-		(color 0 0 0 0)
 	)
 	(junction
@@
 	(wire
 		(pts
-			(xy 148.59 81.28) (xy 148.59 76.2)
-		)
-		(stroke
-			(width 0)
-			(type default)
-		)
-	)
-	(wire
-		(pts
 			(xy 77.47 63.5) (xy 77.47 80.01)
 		)
@@
 	(wire
 		(pts
-			(xy 160.02 83.82) (xy 160.02 81.28)
-		)
-		(stroke
-			(width 0)
-			(type default)
-		)
-	)
-	(wire
-		(pts
 			(xy 77.47 55.88) (xy 77.47 53.34)
 		)
@@
 	(wire
 		(pts
-			(xy 148.59 66.04) (xy 148.59 76.2)
+			(xy 148.59 59.69) (xy 148.59 76.2)
 		)
 		(stroke
@@
 	(wire
 		(pts
-			(xy 148.59 66.04) (xy 163.83 66.04)
-		)
-		(stroke
-			(width 0)
-			(type default)
-		)
-	)
-	(wire
-		(pts
 			(xy 50.8 80.01) (xy 77.47 80.01)
 		)
@@
 	(wire
 		(pts
-			(xy 160.02 81.28) (xy 148.59 81.28)
-		)
-		(stroke
-			(width 0)
-			(type default)
-		)
-	)
-	(wire
-		(pts
 			(xy 148.59 76.2) (xy 163.83 76.2)
 		)
@@
 	(wire
 		(pts
-			(xy 163.83 83.82) (xy 160.02 83.82)
-		)
-		(stroke
-			(width 0)
-			(type default)
-		)
-	)
-	(wire
-		(pts
 			(xy 163.83 78.74) (xy 156.21 78.74)
 		)
@@
 		)
 		(stroke
-			(width 0)
-			(type default)
-		)
-	)
-	(wire
-		(pts
-			(xy 148.59 59.69) (xy 148.59 66.04)
-		)
-		(stroke
