File: moisture/moisture.kicad_sch (KiCad schematic)
At the start: 8 parts, among them U101 FDC1004DGSR, U103 TLV75733PDBV

Commit message: WIP
Parts:
- U101: footprint easyeda2kicad:MSOP-10 -> Package_SO:MSOP-10_3x3mm_P0.5mm
Changed lines of the file:
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@@
 			)
 		)
-		(property "Footprint" "easyeda2kicad:MSOP-10"
+		(property "Footprint" "Package_SO:MSOP-10_3x3mm_P0.5mm"
 			(at 195.58 50.8 0)
 			(effects
@@
 			(effects
 				(font
+					(size 1.27 1.27)
+				)
+				(hide yes)
+			)
+		)
+		(property "Label" ""
+			(at 195.58 63.5 0)
+			(effects
+				(font
