File: leds/UHP500-Conn/UHP600-Conn.kicad_sch (KiCad schematic)
At the start: 15 parts, among them CN1 39288020, CN2 39288020, CN3 39288020, CN4 39288020, J1 428202214, J2 428202214

Commit message: final tweaks
Parts:
- removed H5, H6, H8: MountingHole, MountingHole:MountingHole_3.7mm, symbol Mechanical:MountingHole
- removed H7: MountingHole, MountingHole:MountingHole_3.5mm, symbol Mechanical:MountingHole
- H1, H2, H3, H4: footprint MountingHole:MountingHole_3.5mm_Pad_Via -> MountingHole:MountingHole_4.3mm_M4_Pad_Via
- J1, J2: footprint CONN_SDA-42820-0002_02_RC_MOL -> easyeda2kicad:CONN_SDA-42820-0002_02_RC_MOL
