File: leds/low_profile/low_profile.kicad_pcb (KiCad board)
At the start: 4 copper layers, 94 x 74 mm, 91 parts, among them CN1 39303035, CN10 39-30-1020, CN13 39-30-1020, CN14 39-30-1020, CN2 39303035, CN4 BM04B-SRSS-TB(LF)(SN), CN5 39-30-1020, CN6 39-30-1020, CN9 39-30-1020, J1 Conn_01x06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

Commit message: Low profile LED controller
Parts:
- added C5: C_Polarized, Capacitor_SMD:CP_Elec_8x11.9, F.Cu at (81.8, 54.5)
- added C6: C_Polarized, Capacitor_SMD:CP_Elec_8x11.9, F.Cu at (62.5, 70.0)
- added D6: D_TVS, Diode_SMD:D_SMB, F.Cu at (81.8, 47.5)
- L1: value XGL4040-153MEC -> XAL4040-103MEC; footprint easyeda2kicad:IND-SMD_L4.0-W4.0_XAL4040-103 -> easyeda2kicad:IND-SMD_L4.0-W4.0-A
- moved TP1 25.2 mm to (91.0, 68.0)
- moved L1 0.29 mm to (101.0, 54.3)
Routing:
- net /esp32/LED1: track 77.7 -> 81.7 mm
- net /esp32/EN1: track 70.8 -> 72.8 mm
- net GND: vias 45 -> 77
- net /5V: vias 14 -> 18
Other:
- board text added: "Ada"
- board text added: "Isaac"
- board text added: "JPA041556"
- board text added: "LEDs v0.5"
- board text removed: "LEDs v0.5 low_profile"
