File: leds/power_injection/buck24v.kicad_sch (KiCad schematic)
At the start: 25 parts, among them U1 TPS259474LRPWR, U15 TPSM86837RCGR

Commit message: power injection v0.1
Parts:
- added C15: 15nF, Capacitor_SMD:C_0402_1005Metric, symbol Device:C
- added R10: 100, Resistor_SMD:R_0402_1005Metric, symbol Device:R
- added TP1: TestPoint, TestPoint:TestPoint_Pad_1.0x1.0mm, symbol Connector:TestPoint
- C11: renamed from C42; value 22nF -> 100nF
- R4: renamed from R6; value 73.2k -> 470k
- R5: renamed from R13; value 73.2k -> 45.3k
- R6: renamed from R22; value 73.2k -> 147k
- R7: renamed from R23; value 73.2k -> 562
- R8: renamed from R24; value 73.2k -> 100k
- R9: renamed from R25; value 73.2k -> 34k
- renumbered C34 to C1, C39 to C10, C32 to C12, C26 to C13, C31 to C14, C24 to C2, C38 to C3, C35 to C4, C36 to C5, C37 to C6, C41 to C7, C40 to C8, C33 to C9, R14 to R2, R21 to R3, U15 to U1, U1 to U2
Connections:
- net 5V_RAW: now also TP1.1
- net GND: now also C15.2
- net at U2.7 (DVDT): now also R10.1; no longer C11.1
- net at U2.10 (ITIMER): now also C15.1
- new net: C11.1, R10.2
Other:
- moved on the sheet: C11, R7
