File: leds/strip_small_rgbww/strip_small_rgbww.kicad_pcb (KiCad board)
At the start: 4 copper layers, 295.1 x 12 mm, 123 parts, among them J1 Conn_01x01_Socket, J2 Conn_01x01_Socket, J3 Conn_01x01_Socket, J4 Conn_01x01_Socket, J5 Conn_01x01_Socket, J6 Conn_01x01_Socket, J7 Conn_01x01_Socket, U1 THVD2450DR, U10 TLC59711PWP, U2 TLC59711PWP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

Commit message: update non-standard LED foot prints
Parts:
- D10, D15, D20, D25, D30, D35, D40, D45, D5, D50: footprint LED_SMD:LED_PLCC_2835_Handsoldering -> easyeda2kicad:LED-SMD_L3.5-W2.8-RD-B
- D12, D17, D2, D22, D27, D32, D37, D42, D47, D7: footprint LED_SMD:LED_PLCC_2835_Handsoldering -> easyeda2kicad:LED-SMD_L3.2-W2.8-RD_YELLOW
