File: leds/strip_small_rgbww/untitled.kicad_sch (KiCad schematic)
At the start: 13 parts, among them U2 TLC59711PWP

Commit message: update non-standard LED foot prints
Parts:
- D10, D5: footprint LED_SMD:LED_PLCC_2835_Handsoldering -> easyeda2kicad:LED-SMD_L3.5-W2.8-RD-B
- D2, D7: footprint LED_SMD:LED_PLCC_2835_Handsoldering -> easyeda2kicad:LED-SMD_L3.2-W2.8-RD_YELLOW
Changed lines of the file:
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@@
 			)
 		)
-		(property "Footprint" "LED_SMD:LED_PLCC_2835_Handsoldering"
+		(property "Footprint" "easyeda2kicad:LED-SMD_L3.2-W2.8-RD_YELLOW"
 			(at 200.66 35.56 0)
 			(effects
@@
 			)
 		)
-		(property "Footprint" "LED_SMD:LED_PLCC_2835_Handsoldering"
+		(property "Footprint" "easyeda2kicad:LED-SMD_L3.5-W2.8-RD-B"
 			(at 255.27 35.56 0)
 			(effects
@@
 			)
 		)
-		(property "Footprint" "LED_SMD:LED_PLCC_2835_Handsoldering"
+		(property "Footprint" "easyeda2kicad:LED-SMD_L3.2-W2.8-RD_YELLOW"
 			(at 55.88 34.29 0)
 			(effects
@@
 			)
 		)
-		(property "Footprint" "LED_SMD:LED_PLCC_2835_Handsoldering"
+		(property "Footprint" "easyeda2kicad:LED-SMD_L3.5-W2.8-RD-B"
 			(at 110.49 34.29 0)
 			(effects
