File: leds/high_speed/high_speed.kicad_pcb (KiCad board)
At the start: 4 copper layers, 94 x 74 mm, 89 parts, among them CN1 39-30-1020, CN13 39-30-1020, CN2 39-30-1020, CN3 1053141108, CN4 BM04B-SRSS-TB(LF)(SN), CN5 39-30-1020, J1 Conn_01x06, J2 428202214, Q1 BSS138, Q2 BSS138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

Commit message: high-speed v2.1 fab
Parts:
- added CN6: 39-30-1020, easyeda2kicad:CONN-TH_2P-P5.50_39-30-1020, F.Cu at (80.2, 38.3)
- added TP6: LabeledTestPoint, easyeda2kicad:LabeledTestPoint, F.Cu at (95.0, 39.5)
- added TP7: LabeledTestPoint, easyeda2kicad:LabeledTestPoint, F.Cu at (95.0, 44.8)
- added TP8: LabeledTestPoint, easyeda2kicad:LabeledTestPoint, F.Cu at (95.0, 50.2)
- added TP9: LabeledTestPoint, easyeda2kicad:LabeledTestPoint, F.Cu at (95.0, 55.2)
Connections:
- U1 pad 4: unconnected-(U1-IO4-Pad4) -> /esp32/T1
- U1 pad 5: unconnected-(U1-IO5-Pad5) -> /esp32/T2
- U1 pad 6: unconnected-(U1-IO6-Pad6) -> /esp32/T3
- U1 pad 7: unconnected-(U1-IO7-Pad7) -> /esp32/T4
Routing:
- net /esp32/T4: track 0.00 -> 34.7 mm, vias 0 -> 1
- net /esp32/T3: track 0.00 -> 32.9 mm, vias 0 -> 1
- net /esp32/T2: track 0.00 -> 30.8 mm, vias 0 -> 1
- net /esp32/T1: track 0.00 -> 29.9 mm, vias 0 -> 1
Other:
- board text added: "+24V"
- board text added: "LEDs v2.1"
- board text removed: "LEDs v2.0"
