File: leds/high_speed/led_channel.kicad_sch (KiCad schematic)
At the start: 19 parts, among them CN1 39-30-1020, CN13 39-30-1020, CN2 39-30-1020, CN3 1053141108, CN5 39-30-1020, U19 MP5048GU-Z

Commit message: high-speed v2.1 fab
Parts:
- D3: LCSC Part C151256 -> C178227
Changed lines of the file:
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@@
 			)
 		)
-		(property "LCSC Part" "C151256"
+		(property "LCSC Part" "C178227"
 			(at 199.39 74.93 0)
 			(effects
