File: leds/lamp/3v3.kicad_sch (KiCad schematic)
At the start: 6 parts, among them U4 TPS73733DCQ_C5220270

Commit message: Lamp v0.1 Fabrication
Parts:
- renumbered C15 to C5, C16 to C6, C17 to C7, C18 to C8, R12 to R10, U4 to U2
Changed lines of the file:
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@@
 		(dnp no)
 		(fields_autoplaced yes)
-		(property "Reference" "C16"
+		(property "Reference" "C6"
 			(at 88.9 77.4699 0)
 			(effects
@@
 			(project "espamp"
 				(path "/48ddfdd8-68fa-4e63-aa18-bc113cdf8cfa/ff982210-6c86-422a-a66b-20bff67bd030"
-					(reference "C16")
+					(reference "C6")
 					(unit 1)
 				)
@@
 		(dnp no)
 		(fields_autoplaced yes)
-		(property "Reference" "R12"
+		(property "Reference" "R10"
 			(at 90.17 55.88 90)
 			(effects
@@
 			(project "espamp"
 				(path "/48ddfdd8-68fa-4e63-aa18-bc113cdf8cfa/ff982210-6c86-422a-a66b-20bff67bd030"
-					(reference "R12")
+					(reference "R10")
 					(unit 1)
 				)
@@
 		(dnp no)
 		(fields_autoplaced yes)
-		(property "Reference" "C17"
+		(property "Reference" "C7"
 			(at 119.38 71.1199 0)
 			(effects
@@
 			(project "espamp"
 				(path "/48ddfdd8-68fa-4e63-aa18-bc113cdf8cfa/ff982210-6c86-422a-a66b-20bff67bd030"
-					(reference "C17")
+					(reference "C7")
 					(unit 1)
 				)
@@
 		(on_board yes)
 		(dnp no)
-		(property "Reference" "U4"
+		(property "Reference" "U2"
 			(at 108.712 64.262 0)
 			(effects
@@
 			(project "espamp"
 				(path "/48ddfdd8-68fa-4e63-aa18-bc113cdf8cfa/ff982210-6c86-422a-a66b-20bff67bd030"
-					(reference "U4")
+					(reference "U2")
 					(unit 1)
 				)
@@
 		(dnp no)
 		(fields_autoplaced yes)
-		(property "Reference" "#PWR018"
+		(property "Reference" "#PWR011"
 			(at 110.49 90.17 0)
 			(effects
@@
 			(project ""
 				(path "/48ddfdd8-68fa-4e63-aa18-bc113cdf8cfa/ff982210-6c86-422a-a66b-20bff67bd030"
-					(reference "#PWR018")
+					(reference "#PWR011")
 					(unit 1)
 				)
@@
 		(dnp no)
 		(fields_autoplaced yes)
-		(property "Reference" "C18"
+		(property "Reference" "C8"
 			(at 132.08 71.1199 0)
 			(effects
@@
 			(project "espamp"
 				(path "/48ddfdd8-68fa-4e63-aa18-bc113cdf8cfa/ff982210-6c86-422a-a66b-20bff67bd030"
-					(reference "C18")
+					(reference "C8")
 					(unit 1)
 				)
@@
 		(dnp no)
 		(fields_autoplaced yes)
-		(property "Reference" "C15"
+		(property "Reference" "C5"
 			(at 78.74 71.1199 0)
 			(effects
@@
 			(project "espamp"
 				(path "/48ddfdd8-68fa-4e63-aa18-bc113cdf8cfa/ff982210-6c86-422a-a66b-20bff67bd030"
-					(reference "C15")
-					(unit 1)
-				)
+					(reference "C5")
+					(unit 1)
+				)
