File: leds/lamp/lamp.kicad_pcb (KiCad board)
At the start: 4 copper layers, 94 x 74 mm, 44 parts, among them CN4 BM04B-SRSS-TB(LF)(SN), J1 Conn_01x06, Q1 BSS138, Q2 BSS138, SW1 EVPAA602W, SW3 EVPAA602W, U1 ESP32-S3-WROOM-1, U19 MP5048GU-Z, U4 TPS73733DCQ_C5220270, U5 ADS1115IDGSR

Commit message: WIP: Lamp
Parts:
- added C10: 10uF, Capacitor_SMD:C_0603_1608Metric, F.Cu at (48.8, 29.2)
- added C11: 10uF, Capacitor_SMD:C_0603_1608Metric, F.Cu at (42.2, 30.2)
- added C12: 1uF, Capacitor_SMD:C_0603_1608Metric, F.Cu at (42.2, 28.8)
- added C13: 330uF, easyeda2kicad:CAP-SMD_L7.3-W4.3-FD, F.Cu at (34.0, 23.2)
- added C14: 100nF, Capacitor_SMD:C_0603_1608Metric, F.Cu at (70.5, 75.2)
- added C5: 10uF, Capacitor_SMD:C_0603_1608Metric, F.Cu at (42.1, 42.5)
- added C6: 100nF, Capacitor_SMD:C_0603_1608Metric, F.Cu at (42.1, 44.0)
- added C8: 1uF, Capacitor_SMD:C_0603_1608Metric, F.Cu at (63.0, 41.5)
- added C9: 1uF, Capacitor_SMD:C_0603_1608Metric, F.Cu at (47.2, 29.2)
- added F1: Fuse, easyeda2kicad:FUSE-SMD_L9.8-W5.0_01550900M, F.Cu at (28.8, 71.2)
- added J2: Conn_02x05_Top_Bottom, Connector_Molex:Molex_Nano-Fit_105310-xx10_2x05_P2.50mm_Vertical, F.Cu at (35.2, 38.0)
- added J3: Conn_01x02, Connector_Molex:Molex_Nano-Fit_105309-xx02_1x02_P2.50mm_Vertical, F.Cu at (37.1, 45.2)
- added J4: Conn_01x02, Connector_Molex:Molex_Nano-Fit_105309-xx02_1x02_P2.50mm_Vertical, F.Cu at (69.6, 38.8)
- added J5: Conn_01x04, Connector_Molex:Molex_Nano-Fit_105310-xx04_2x02_P2.50mm_Vertical, F.Cu at (70.3, 28.2)
- added J6: Conn_01x02, Connector_Molex:Molex_Mini-Fit_Jr_5569-02A2_2x01_P4.20mm_Horizontal, F.Cu at (25.1, 57.8)
- added J7: Conn_01x02, Connector_Molex:Molex_Nano-Fit_105309-xx02_1x02_P2.50mm_Vertical, F.Cu at (23.0, 38.8)
- added PS1: IRM-20-5, Converter_ACDC:Converter_ACDC_MeanWell_IRM-20-xx_THT, B.Cu at (62.5, 70.8)
- added R15: 10k, Resistor_SMD:R_0805_2012Metric, F.Cu at (70.7, 35.0)
- added R16: 1.5k, Resistor_SMD:R_0603_1608Metric, F.Cu at (41.2, 22.0)
- added R6: 1k, Resistor_SMD:R_0603_1608Metric, F.Cu at (25.0, 31.8)
- added R7: 634kΩ, Resistor_SMD:R_0603_1608Metric, F.Cu at (45.6, 45.5)
- added R8: R, Resistor_SMD:R_0805_2012Metric, F.Cu at (45.9, 49.5)
- added R9: R, Resistor_SMD:R_0805_2012Metric, F.Cu at (45.9, 47.5)
- added RV1: Varistor, Varistor:RV_Disc_D12mm_W7.5mm_P7.5mm, F.Cu at (34.6, 56.4)
- added TP1: TestPoint, TestPoint:TestPoint_Pad_D1.0mm, F.Cu at (48.8, 22.8)
- added TP2: TestPoint, TestPoint:TestPoint_Pad_D1.0mm, F.Cu at (50.8, 22.8)
- added TP3: TestPoint, TestPoint:TestPoint_Pad_D1.0mm, F.Cu at (43.2, 22.2)
- added U2: MAX98357A, Package_DFN_QFN:TQFN-16-1EP_3x3mm_P0.5mm_EP1.23x1.23mm, F.Cu at (41.8, 46.9)
- added U3: LM73100RPWR, easyeda2kicad:VQFN-10_L2.0-W2.0-P0.45-TL, F.Cu at (46.0, 24.0)
- added U6: ICS-43434_C5656610, easyeda2kicad:MIC-SMD_6P-L3.5-W2.7-P0.90-BL, F.Cu at (70.8, 71.5)
- U19: value MP5048GU-Z -> MP5048AGU-Z
- moved H1 200.0 mm to (24.0, 24.0)
- moved H3 189.4 mm to (24.0, 79.0)
- moved Q2 173.4 mm to (55.6, 28.1), turned to 90 degrees
- moved CN4 168.5 mm to (58.9, 23.5), turned to 0 degrees
- moved R10 168.2 mm to (58.4, 27.6), turned to 90 degrees
- moved R11 164.7 mm to (60.1, 27.6), turned to 90 degrees
- moved Q1 159.6 mm to (62.6, 28.1), turned to 90 degrees
- moved D4 158.8 mm to (26.5, 31.8), turned to 90 degrees
- moved H2 158.0 mm to (79.0, 24.0)
- moved J1 155.7 mm to (59.9, 80.2), turned to 90 degrees
- moved C19 145.6 mm to (60.8, 37.8)
- moved C20 145.6 mm to (60.8, 39.2)
- moved U5 145.6 mm to (59.8, 43.8)
- moved H4 143.2 mm to (79.0, 79.0)
- moved C21 138.3 mm to (52.0, 36.7)
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Connections:
- net /3v3/3v3 renamed /3V3
- U19 pad 1: /led_channel/5V -> /5V
- U19 pad 18: /led_channel/5V -> /5V
- U19 pad 2: /led_channel/5V -> /5V
- U5 pad 6: /a2d/AIN3 -> /10k_temp/OUT
Routing:
- net Net-(PS1-AC/L): track 0.00 -> 44.8 mm
- net /esp32/LEDCLOCK: track 0.00 -> 34.8 mm, vias 0 -> 1
- net /esp32/LEDDATA: track 0.00 -> 31.7 mm, vias 0 -> 1
- net Net-(J6-Pin_2): track 0.00 -> 29.9 mm
- net /speaker/I2S.LRCLK: track 0.00 -> 23.1 mm, vias 0 -> 1
- net /speaker/I2S.BCLK: track 0.00 -> 21.8 mm, vias 0 -> 1
- net /speaker/I2S.DIN: track 0.00 -> 21.0 mm, vias 0 -> 1
- net /esp32/Fault: track 1.74 -> 20.2 mm
- net /esp32/SEN: track 0.00 -> 18.3 mm, vias 0 -> 1
- net Net-(J6-Pin_1): track 0.00 -> 15.5 mm
- net /a2d/I2C.SDA: track 2.65 -> 17.6 mm, vias 0 -> 1
- net /a2d/I2C.SCL: track 2.51 -> 17.0 mm, vias 0 -> 1
- net GND: track 11.1 -> 24.2 mm, vias 12 -> 30
- net /3V3: track 7.23 -> 0.00 mm, vias 1 -> 6
- net /5V: track 15.9 -> 9.43 mm, vias 2 -> 9
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- added copper zone on F.Cu, net /3V3
- added copper zone on F.Cu, net /5V
- added copper zone on F.Cu, net /dioed/VIN
- added copper zone on F.Cu, net /led_channel/VLED
- removed copper zone on In2.Cu, net /5V
Other:
- board size 94 x 74 mm -> 63 x 63 mm
- board text added: "5V"
- board text added: "AC-IN"
- board text added: "CLK"
- board text added: "DANGER:120VAC"
- board text added: "DIO"
- board text added: "G"
- board text added: "L"
- board text added: "N"
- board text added: "PWR"
- board text added: "S+"
- board text added: "S-"

Commit message: Lamp v0.1 Fabrication
Parts:
- moved U6 9.23 mm to (80.0, 72.2), turned to 90 degrees
- moved C18 7.61 mm to (77.8, 73.0), turned to 90 degrees
- moved J1 3.91 mm to (26.0, 36.2), turned to 0 degrees
- moved SW2 1.76 mm to (74.8, 68.0)
- moved R14 1.59 mm to (69.2, 35.5), turned to 0 degrees
- moved D1 1.21 mm to (80.8, 65.8)
- moved R7 1.21 mm to (80.8, 67.2)
- moved C20 1.10 mm to (48.0, 32.5)
- moved C21 0.56 mm to (48.0, 35.5)
- moved C3 0.14 mm to (78.3, 34.2)
- renumbered C6 to C10, C19 to C11, C20 to C12, C8 to C13, C10 to C14, C9 to C15, C12 to C16, C11 to C17, C14 to C18, C24 to C19, C23 to C20, C22 to C21, C21 to C22, C7 to C23, C13 to C24, C15 to C5, C16 to C6, C17 to C7, C18 to C8, C5 to C9, CN4 to CN1, D4 to D2, J7 to J1, J6 to J2, J5 to J3, J1 to J4, J3 to J5, J4 to J6, J2 to J7, R12 to R10, R9 to R11, R8 to R12, R7 to R13, R15 to R14, R16 to R15, R6 to R16, R13 to R17, R14 to R18, R18 to R19, R22 to R5, R21 to R6, R5 to R7, R10 to R8, R11 to R9, SW3 to SW2, TP3 to TP1, TP1 to TP2, TP2 to TP3, U4 to U2, U5 to U3, U2 to U4, U3 to U5, U19 to U7
Connections:
- C18 pad 1: /mic/3v3 -> /3V3
- J1 pad 1: unconnected-(J7-Pin_1-Pad1) -> /5V
- J1 pad 2: unconnected-(J7-Pin_2-Pad2) -> GND
- U1 pad 12: unconnected-(U1-IO8-Pad12) -> /esp32/Fault
- U1 pad 21: /esp32/Fault -> /esp32/SEN
- U1 pad 22: unconnected-(U1-IO14-Pad22) -> /esp32/I2S.DIN
- U1 pad 23: unconnected-(U1-IO21-Pad23) -> /esp32/I2S.BCLK
- U1 pad 24: unconnected-(U1-IO47-Pad24) -> /esp32/I2S.LRCLK
- U1 pad 25: unconnected-(U1-IO48-Pad25) -> /esp32/I2S.DOUT
- U4 pad 1: /speaker/I2S.DIN -> /esp32/I2S.DIN
- U4 pad 14: /speaker/I2S.LRCLK -> /esp32/I2S.LRCLK
- U4 pad 16: /speaker/I2S.BCLK -> /esp32/I2S.BCLK
- U6 pad 1: /mic/I2S.LRCLK -> /esp32/I2S.LRCLK
- U6 pad 4: /mic/I2S.BCLK -> /esp32/I2S.BCLK
- U6 pad 5: /mic/3v3 -> /3V3
- U6 pad 6: /mic/I2S.DOUT -> /esp32/I2S.DOUT
Routing:
- net /esp32/I2S.LRCLK: track 0.00 -> 54.4 mm, vias 0 -> 3
- net /esp32/I2S.BCLK: track 0.00 -> 50.4 mm, vias 0 -> 3
- net Net-(J4-Pin_6): track 0.00 -> 47.5 mm, vias 0 -> 2
- net /esp32/EN1: track 1.60 -> 38.7 mm, vias 1 -> 2
- net Net-(J4-Pin_5): track 0.00 -> 32.2 mm, vias 0 -> 2
- net /esp32/Fault: track 20.2 -> 51.6 mm, vias 1 -> 3
- net /esp32/T2: track 0.00 -> 29.0 mm, vias 0 -> 1
- net /esp32/I2S.DOUT: track 0.00 -> 26.4 mm, vias 0 -> 2
- net /3V3: track 0.00 -> 26.2 mm, vias 6 -> 14
- net /a2d/AIN1: track 1.17 -> 27.1 mm, vias 1 -> 2
- net /esp32/I2S.DIN: track 0.00 -> 24.9 mm, vias 0 -> 2
- net /esp32/T1: track 0.00 -> 23.9 mm, vias 0 -> 1
- net Net-(J4-Pin_3): track 0.00 -> 23.1 mm
- net /speaker/I2S.LRCLK: track 23.1 -> 0.00 mm, vias 1 -> 0
- net /speaker/I2S.BCLK: track 21.8 -> 0.00 mm, vias 1 -> 0
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- added copper zone on In2.Cu, net /3V3
- added copper zone on In2.Cu, net /5V
- added copper zone on F.Cu, net Net-(U7-VCC)
Other:
- board text added: "Lamp v0.1"
- board text added: "SCL"
- board text added: "SDA"
- board text added: "T"
- board text added: "T2 T1 T4 T3"
- board text added: "VIN"
