File: leds/lamp/led_channel.kicad_sch (KiCad schematic)
At the start: 12 parts, among them J2 Conn_02x05_Top_Bottom, U19 MP5048AGU-Z

Commit message: WIP: Lamp
Parts:
- added C13: 330uF, easyeda2kicad:CAP-SMD_L7.3-W4.3-FD, symbol Device:C_Polarized
Connections:
- net GND: now also C13.2
- net VLED: now also C13.1
Other:
- moved on the sheet: J2
Changed lines of the file:
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@@
 	)
 	(junction
-		(at 264.16 74.93)
+		(at 267.97 74.93)
 		(diameter 0)
 		(color 0 0 0 0)
@@
 	)
 	(junction
-		(at 246.38 69.85)
+		(at 250.19 69.85)
 		(diameter 0)
 		(color 0 0 0 0)
@@
 	)
 	(junction
-		(at 246.38 74.93)
+		(at 250.19 74.93)
 		(diameter 0)
 		(color 0 0 0 0)
@@
 	)
 	(junction
-		(at 264.16 72.39)
+		(at 267.97 72.39)
+		(diameter 0)
+		(color 0 0 0 0)
+	)
+	(junction
+		(at 240.03 101.6)
 		(diameter 0)
 		(color 0 0 0 0)
@@
 	)
 	(junction
-		(at 264.16 77.47)
+		(at 267.97 77.47)
 		(diameter 0)
 		(color 0 0 0 0)
@@
 	)
 	(junction
-		(at 246.38 72.39)
+		(at 240.03 69.85)
+		(diameter 0)
+		(color 0 0 0 0)
+	)
+	(junction
+		(at 250.19 72.39)
 		(diameter 0)
 		(color 0 0 0 0)
@@
 	(wire
 		(pts
-			(xy 264.16 74.93) (xy 264.16 77.47)
+			(xy 267.97 74.93) (xy 267.97 77.47)
 		)
 		(stroke
@@
 	(wire
 		(pts
+			(xy 240.03 69.85) (xy 250.19 69.85)
+		)
+		(stroke
+			(width 0)
+			(type default)
+		)
+	)
+	(wire
+		(pts
 			(xy 209.55 101.6) (xy 199.39 101.6)
 		)
@@
 	(wire
 		(pts
-			(xy 264.16 69.85) (xy 264.16 72.39)
+			(xy 267.97 69.85) (xy 267.97 72.39)
 		)
 		(stroke
@@
 	(wire
 		(pts
-			(xy 261.62 67.31) (xy 264.16 67.31)
+			(xy 265.43 67.31) (xy 267.97 67.31)
 		)
 		(stroke
@@
 	(wire
 		(pts
+			(xy 196.85 69.85) (xy 240.03 69.85)
+		)
+		(stroke
+			(width 0)
+			(type default)
+		)
+	)
+	(wire
+		(pts
 			(xy 125.73 76.2) (xy 129.54 76.2)
 		)
@@
 	(wire
 		(pts
+			(xy 240.03 101.6) (xy 267.97 101.6)
+		)
+		(stroke
+			(width 0)
+			(type default)
+		)
+	)
+	(wire
+		(pts
 			(xy 196.85 90.17) (xy 199.39 90.17)
 		)
@@
 	(wire
 		(pts
-			(xy 261.62 72.39) (xy 264.16 72.39)
+			(xy 265.43 72.39) (xy 267.97 72.39)
 		)
 		(stroke
@@
 	(wire
 		(pts
-			(xy 261.62 77.47) (xy 264.16 77.47)
+			(xy 265.43 77.47) (xy 267.97 77.47)
 		)
 		(stroke
@@
 	(wire
 		(pts
-			(xy 248.92 74.93) (xy 246.38 74.93)
+			(xy 252.73 74.93) (xy 250.19 74.93)
 		)
 		(stroke
@@
 	(wire
 		(pts
-			(xy 246.38 77.47) (xy 246.38 74.93)
+			(xy 250.19 77.47) (xy 250.19 74.93)
 		)
 		(stroke
@@
 	(wire
 		(pts
-			(xy 261.62 74.93) (xy 264.16 74.93)
-		)
-		(stroke
-			(width 0)
-			(type default)
-		)
-	)
-	(wire
-		(pts
-			(xy 264.16 77.47) (xy 264.16 101.6)
-		)
-		(stroke
-			(width 0)
-			(type default)
-		)
-	)
-	(wire
-		(pts
-			(xy 264.16 101.6) (xy 228.6 101.6)
-		)
-		(stroke
-			(width 0)
-			(type default)
-		)
-	)
-	(wire
-		(pts
-			(xy 248.92 72.39) (xy 246.38 72.39)
-		)
-		(stroke
-			(width 0)
-			(type default)
-		)
-	)
-	(wire
-		(pts
-			(xy 248.92 77.47) (xy 246.38 77.47)
+			(xy 265.43 74.93) (xy 267.97 74.93)
+		)
+		(stroke
+			(width 0)
+			(type default)
+		)
+	)
+	(wire
+		(pts
+			(xy 267.97 77.47) (xy 267.97 101.6)
+		)
+		(stroke
+			(width 0)
+			(type default)
+		)
+	)
+	(wire
+		(pts
+			(xy 252.73 72.39) (xy 250.19 72.39)
+		)
+		(stroke
+			(width 0)
+			(type default)
+		)
+	)
+	(wire
+		(pts
+			(xy 252.73 77.47) (xy 250.19 77.47)
 		)
 		(stroke
@@
 	(wire
 		(pts
-			(xy 246.38 72.39) (xy 246.38 69.85)
+			(xy 228.6 101.6) (xy 240.03 101.6)
+		)
+		(stroke
+			(width 0)
+			(type default)
+		)
+	)
+	(wire
+		(pts
+			(xy 250.19 72.39) (xy 250.19 69.85)
 		)
 		(stroke
@@
 	(wire
 		(pts
-			(xy 196.85 69.85) (xy 246.38 69.85)
-		)
-		(stroke
-			(width 0)
-			(type default)
-		)
-	)
-	(wire
-		(pts
 			(xy 147.32 72.39) (xy 147.32 76.2)
 		)
@@
 	(wire
 		(pts
-			(xy 246.38 74.93) (xy 246.38 72.39)
-		)
-		(stroke
-			(width 0)
-			(type default)
-		)
-	)
-	(wire
-		(pts
-			(xy 261.62 69.85) (xy 264.16 69.85)
+			(xy 250.19 74.93) (xy 250.19 72.39)
+		)
+		(stroke
+			(width 0)
+			(type default)
+		)
+	)
+	(wire
+		(pts
+			(xy 265.43 69.85) (xy 267.97 69.85)
 		)
 		(stroke
@@
 	(wire
 		(pts
-			(xy 246.38 67.31) (xy 248.92 67.31)
-		)
-		(stroke
-			(width 0)
-			(type default)
-		)
-	)
-	(wire
-		(pts
-			(xy 246.38 69.85) (xy 248.92 69.85)
+			(xy 250.19 67.31) (xy 252.73 67.31)
+		)
+		(stroke
+			(width 0)
+			(type default)
+		)
+	)
+	(wire
+		(pts
+			(xy 250.19 69.85) (xy 252.73 69.85)
 		)
 		(stroke
@@
 	(wire
 		(pts
-			(xy 264.16 72.39) (xy 264.16 74.93)
+			(xy 240.03 77.47) (xy 240.03 101.6)
+		)
+		(stroke
+			(width 0)
+			(type default)
+		)
+	)
+	(wire
+		(pts
+			(xy 267.97 72.39) (xy 267.97 74.93)
 		)
 		(stroke
@@
 	(hierarchical_label "DIN"
 		(shape input)
-		(at 246.38 67.31 180)
+		(at 250.19 67.31 180)
 		(effects
 			(font
@@
 	(hierarchical_label "CLK"
 		(shape input)
-		(at 264.16 67.31 0)
+		(at 267.97 67.31 0)
 		(effects
 			(font
@@
 	(symbol
 		(lib_id "Connector_Generic:Conn_02x05_Top_Bottom")
-		(at 254 72.39 0)
+		(at 257.81 72.39 0)
 		(unit 1)
 		(exclude_from_sim no)
@@
 		(fields_autoplaced yes)
 		(property "Reference" "J2"
-			(at 255.27 60.96 0)
+			(at 259.08 60.96 0)
 			(effects
 				(font
@@
 		)
 		(property "Value" "Conn_02x05_Top_Bottom"
-			(at 255.27 63.5 0)
+			(at 259.08 63.5 0)
 			(effects
 				(font
@@
 		)
 		(property "Footprint" "Connector_Molex:Molex_Nano-Fit_105310-xx10_2x05_P2.50mm_Vertical"
-			(at 254 72.39 0)
+			(at 257.81 72.39 0)
 			(effects
 				(font
@@
 		)
 		(property "Datasheet" "~"
-			(at 254 72.39 0)
+			(at 257.81 72.39 0)
 			(effects
 				(font
@@
 		)
 		(property "Description" "Generic connector, double row, 02x05, top/bottom pin numbering scheme (row 1: 1...pins_per_row, row2: pins_per_row+1 ... num_pins), script generated (kicad-library-utils/schlib/autogen/connector/)"
-			(at 254 72.39 0)
+			(at 257.81 72.39 0)
 			(effects
 				(font
@@
 		)
 		(property "LCSC Part" "C561763"
-			(at 254 72.39 0)
+			(at 257.81 72.39 0)
 			(effects
 				(font
@@
 					(unit 1)
 				)
+			)
+		)
+	)
+	(symbol
+		(lib_id "Device:C_Polarized")
+		(at 240.03 73.66 0)
+		(unit 1)
+		(exclude_from_sim no)
+		(in_bom yes)
+		(on_board yes)
+		(dnp no)
+		(property "Reference" "C13"
+			(at 244.856 71.882 0)
+			(effects
+				(font
+					(size 1.27 1.27)
+				)
+				(justify left)
+			)
+		)
+		(property "Value" "330uF"
+			(at 243.84 73.914 0)
+			(effects
+				(font
+					(size 1.27 1.27)
+				)
+				(justify left)
+			)
+		)
+		(property "Footprint" "easyeda2kicad:CAP-SMD_L7.3-W4.3-FD"
+			(at 240.9952 77.47 0)
+			(effects
+				(font
+					(size 1.27 1.27)
+				)
+				(hide yes)
+			)
+		)
+		(property "Datasheet" "~"
+			(at 240.03 73.66 0)
+			(effects
+				(font
+					(size 1.27 1.27)
+				)
+				(hide yes)
+			)
+		)
+		(property "Description" "Polarized capacitor"
+			(at 240.03 73.66 0)
+			(effects
+				(font
+					(size 1.27 1.27)
+				)
+				(hide yes)
+			)
+		)
+		(property "LCSC Part" "C2159214"
+			(at 240.03 83.82 0)
+			(effects
+				(font
+					(size 1.27 1.27)
+				)
+				(hide yes)
+			)
+		)
+		(property "Label" ""
+			(at 240.03 73.66 0)
+			(effects
+				(font
+					(size 1.27 1.27)
+				)
+				(hide yes)
+			)
+		)
+		(pin "1"
+		)
+		(pin "2"
+		)
+		(instances
+			(project "lamp"
+				(path "/48ddfdd8-68fa-4e63-aa18-bc113cdf8cfa/f2bbebe1-7e19-419b-a0b6-59692ffc8a76"
+					(reference "C13")
+					(unit 1)
+				)

Commit message: Lamp v0.1 Fabrication
Parts:
- renumbered C24 to C19, C23 to C20, C22 to C21, C21 to C22, C7 to C23, C13 to C24, D4 to D2, J2 to J7, R6 to R16, R13 to R17, R14 to R18, R18 to R19, U19 to U7
Changed lines of the file:
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@@
 		(dnp no)
 		(fields_autoplaced yes)
-		(property "Reference" "J2"
+		(property "Reference" "J7"
 			(at 259.08 60.96 0)
 			(effects
@@
 			(project "lamp"
 				(path "/48ddfdd8-68fa-4e63-aa18-bc113cdf8cfa/f2bbebe1-7e19-419b-a0b6-59692ffc8a76"
-					(reference "J2")
+					(reference "J7")
 					(unit 1)
 				)
@@
 		(dnp no)
 		(fields_autoplaced yes)
-		(property "Reference" "U19"
+		(property "Reference" "U7"
 			(at 185.42 59.69 0)
 			(effects
@@
 			(project "high_speed"
 				(path "/48ddfdd8-68fa-4e63-aa18-bc113cdf8cfa/f2bbebe1-7e19-419b-a0b6-59692ffc8a76"
-					(reference "U19")
+					(reference "U7")
 					(unit 1)
 				)
@@
 		(dnp no)
 		(fields_autoplaced yes)
-		(property "Reference" "#PWR01"
+		(property "Reference" "#PWR017"
 			(at 185.42 107.95 0)
 			(effects
@@
 			(project ""
 				(path "/48ddfdd8-68fa-4e63-aa18-bc113cdf8cfa/f2bbebe1-7e19-419b-a0b6-59692ffc8a76"
-					(reference "#PWR01")
+					(reference "#PWR017")
 					(unit 1)
 				)
@@
 		(dnp no)
 		(fields_autoplaced yes)
-		(property "Reference" "R14"
+		(property "Reference" "R18"
 			(at 161.29 90.1699 0)
 			(effects
@@
 			(project ""
 				(path "/48ddfdd8-68fa-4e63-aa18-bc113cdf8cfa/f2bbebe1-7e19-419b-a0b6-59692ffc8a76"
-					(reference "R14")
+					(reference "R18")
 					(unit 1)
 				)
@@
 		(dnp no)
 		(fields_autoplaced yes)
-		(property "Reference" "C24"
+		(property "Reference" "C19"
 			(at 140.97 87.6299 0)
 			(effects
@@
 			(project "high_speed"
 				(path "/48ddfdd8-68fa-4e63-aa18-bc113cdf8cfa/f2bbebe1-7e19-419b-a0b6-59692ffc8a76"
-					(reference "C24")
+					(reference "C19")
 					(unit 1)
 				)
@@
 		(on_board yes)
 		(dnp no)
-		(property "Reference" "C13"
+		(property "Reference" "C24"
 			(at 244.856 71.882 0)
 			(effects
@@
 			(project "lamp"
 				(path "/48ddfdd8-68fa-4e63-aa18-bc113cdf8cfa/f2bbebe1-7e19-419b-a0b6-59692ffc8a76"
-					(reference "C13")
+					(reference "C24")
 					(unit 1)
 				)
@@
 		(dnp no)
 		(fields_autoplaced yes)
-		(property "Reference" "R13"
+		(property "Reference" "R17"
 			(at 152.4 87.6299 0)
 			(effects
@@
 			(project ""
 				(path "/48ddfdd8-68fa-4e63-aa18-bc113cdf8cfa/f2bbebe1-7e19-419b-a0b6-59692ffc8a76"
-					(reference "R13")
+					(reference "R17")
 					(unit 1)
 				)
@@
 		(dnp no)
 		(fields_autoplaced yes)
-		(property "Reference" "C21"
+		(property "Reference" "C22"
 			(at 222.25 85.0899 0)
 			(effects
@@
 			(project ""
 				(path "/48ddfdd8-68fa-4e63-aa18-bc113cdf8cfa/f2bbebe1-7e19-419b-a0b6-59692ffc8a76"
-					(reference "C21")
+					(reference "C22")
 					(unit 1)
 				)
@@
 		(dnp no)
 		(fields_autoplaced yes)
-		(property "Reference" "C22"
+		(property "Reference" "C21"
 			(at 213.36 90.1699 0)
 			(effects
@@
 			(project ""
 				(path "/48ddfdd8-68fa-4e63-aa18-bc113cdf8cfa/f2bbebe1-7e19-419b-a0b6-59692ffc8a76"
-					(reference "C22")
+					(reference "C21")
 					(unit 1)
 				)
@@
 		(dnp no)
 		(fields_autoplaced yes)
-		(property "Reference" "R18"
+		(property "Reference" "R19"
 			(at 170.18 92.7099 0)
 			(effects
@@
 			(project ""
 				(path "/48ddfdd8-68fa-4e63-aa18-bc113cdf8cfa/f2bbebe1-7e19-419b-a0b6-59692ffc8a76"
-					(reference "R18")
+					(reference "R19")
 					(unit 1)
 				)
@@
 		(dnp no)
 		(fields_autoplaced yes)
-		(property "Reference" "C23"
+		(property "Reference" "C20"
 			(at 203.2 92.7099 0)
 			(effects
@@
 			(project ""
 				(path "/48ddfdd8-68fa-4e63-aa18-bc113cdf8cfa/f2bbebe1-7e19-419b-a0b6-59692ffc8a76"
-					(reference "C23")
+					(reference "C20")
 					(unit 1)
 				)
@@
 		(dnp no)
 		(fields_autoplaced yes)
-		(property "Reference" "R6"
+		(property "Reference" "R16"
 			(at 133.35 69.85 90)
 			(effects
@@
 			(project "high_speed"
 				(path "/48ddfdd8-68fa-4e63-aa18-bc113cdf8cfa/f2bbebe1-7e19-419b-a0b6-59692ffc8a76"
-					(reference "R6")
+					(reference "R16")
 					(unit 1)
 				)
@@
 		(dnp no)
 		(fields_autoplaced yes)
-		(property "Reference" "C7"
+		(property "Reference" "C23"
 			(at 232.41 82.5499 0)
 			(effects
@@
 			(project ""
 				(path "/48ddfdd8-68fa-4e63-aa18-bc113cdf8cfa/f2bbebe1-7e19-419b-a0b6-59692ffc8a76"
-					(reference "C7")
+					(reference "C23")
 					(unit 1)
 				)
@@
 		(dnp no)
 		(fields_autoplaced yes)
-		(property "Reference" "D4"
+		(property "Reference" "D2"
 			(at 142.5575 68.58 0)
 			(effects
@@
 			(project "high_speed"
 				(path "/48ddfdd8-68fa-4e63-aa18-bc113cdf8cfa/f2bbebe1-7e19-419b-a0b6-59692ffc8a76"
-					(reference "D4")
-					(unit 1)
-				)
+					(reference "D2")
+					(unit 1)
+				)
